File: mousekey/mousekey_v0p1/ADB_Ports.kicad_sch (KiCad schematic)
At the start: 0 parts

Commit message: Added ADB and Teensy
Parts:
- added J3, J4: MD-40S, CUI_MD-40S, symbol MD-40S:MD-40S
- added JP13, JP14: Jumper_2_Bridged, Connector_PinHeader_2.54mm:PinHeader_1x02_P2.54mm_Vertical, symbol Jumper:Jumper_2_Bridged
- added JP15, JP16, JP17, JP18, JP19, JP20, JP21, JP22: SolderJumper_2_Bridged, Jumper:SolderJumper-2_P1.3mm_Bridged_RoundedPad1.0x1.5mm, symbol Jumper:SolderJumper_2_Bridged
- added R2: 0 ohm, Resistor_SMD:R_0805_2012Metric, symbol Device:R_Small
- added TP1, TP2, TP3, TP4, TP5, TP6, TP7, TP8: TestPoint, TestPoint:TestPoint_THTPad_2.0x2.0mm_Drill1.0mm, symbol Connector:TestPoint
- added U3: LSF0204DPWR, SOP65P640X120-14N, symbol LSF0204DPWR:LSF0204DPWR
Connections:
- new net: J3.8, JP18.2 (B)
- new net: R2.2, U3.8 (~EN)
- new net: JP14.2 (B), JP21.1 (A)
- new net: J4.6, JP21.2 (B)
- new net: J4.3, JP19.2 (B)
- new net: J4.5, JP20.2 (B)
- new net: J4.8, JP22.2 (B)
- new net: J3.5, JP16.2 (B)
- new net: JP13.2 (B), JP17.1 (A)
- new net: J3.3, JP15.2 (B)
- new net: J3.6, JP17.2 (B)
- new net +3V3: U3.1 (VREF_A)
- new net +5V: JP13.1 (A), JP14.1 (A), U3.14 (VREF_B)
- new net ADB_A_Data: JP15.1 (A), TP5.1, U3.13 (B1)
- new net ADB_A_PWR: JP16.1 (A), TP6.1, U3.12 (B2)
- new net ADB_B_Data: JP19.1 (A), TP7.1, U3.11 (B3)
- new net ADB_B_PWR: JP20.1 (A), TP8.1, U3.10 (B4)
- new net GND: J3.S1 (SHIELD), J4.S1 (SHIELD), JP18.1 (A), JP22.1 (A), R2.1, U3.7 (GND)
- new net TTL_ADB_A_Data: TP1.1, U3.2 (A1)
- new net TTL_ADB_A_PWR: TP2.1, U3.3 (A2)
- new net TTL_ADB_B_Data: TP3.1, U3.4 (A3)
- new net TTL_ADB_B_PWR: TP4.1, U3.5 (A4)
