File: mousekey/mousekey_v0p1/mousekey_v0p1.kicad_pcb (KiCad board)
At the start: 2 copper layers, 95 x 69.7 mm, 46 parts, among them J1 MD-60S, J2 MD-60S, J3 MD-40S, J4 MD-40S, U1 LSF0204DPWR, U3 LSF0204DPWR

Commit message: updates
Parts:
- added U2: Teensy4.1, teensy:Teensy41, F.Cu at (118.5, 85.8)
- added U4: CY7C65634-48AXCT, teensy:CY7C65634-48AXCT, F.Cu at (154.5, 70.3)

Commit message: updates
Parts:
- added C1: 0.1u, Capacitor_SMD:C_1206_3216Metric, F.Cu at (152.9, 82.4)
- added C2: 20p, Capacitor_SMD:C_1206_3216Metric, F.Cu at (150.1, 71.5)
- added C3: 0.1u, Capacitor_SMD:C_1206_3216Metric, F.Cu at (152.9, 79.5)
- added C4: 0.1u, Capacitor_SMD:C_1206_3216Metric, F.Cu at (152.9, 76.7)
- added C5: 20p, Capacitor_SMD:C_1206_3216Metric, F.Cu at (145.5, 71.5)
- added C6: 0.1u, Capacitor_SMD:C_1206_3216Metric, F.Cu at (140.8, 71.5)
- added C7: 0.1u, Capacitor_SMD:C_1206_3216Metric, F.Cu at (137.0, 81.3)
- added C8: 0.1u, Capacitor_SMD:C_1206_3216Metric, F.Cu at (147.0, 87.8)
- added D1: PGB1010603MR, Diode_SMD:D_0201_0603Metric, F.Cu at (163.6, 93.4)
- added D2: PGB1010603MR, Diode_SMD:D_0201_0603Metric, F.Cu at (116.1, 102.2)
- added D3: PGB1010603MR, Diode_SMD:D_0201_0603Metric, F.Cu at (121.5, 102.2)
- added D4: PGB1010603MR, Diode_SMD:D_0201_0603Metric, F.Cu at (163.7, 75.8)
- added D5: PGB1010603MR, Diode_SMD:D_0201_0603Metric, F.Cu at (163.5, 85.6)
- added D6: PGB1010603MR, Diode_SMD:D_0201_0603Metric, F.Cu at (163.5, 67.8)
- added J5: USB_A, Connector_USB:USB_A_Molex_67643_Horizontal, F.Cu at (168.4, 74.9)
- added J6: USB_A, Connector_USB:USB_A_Molex_67643_Horizontal, F.Cu at (168.4, 92.7)
- added TP17: TestPoint, TestPoint:TestPoint_THTPad_2.0x2.0mm_Drill1.0mm, F.Cu at (163.5, 70.4)
- added TP18: TestPoint, TestPoint:TestPoint_THTPad_2.0x2.0mm_Drill1.0mm, F.Cu at (163.5, 73.5)
- added TP19: TestPoint, TestPoint:TestPoint_THTPad_2.0x2.0mm_Drill1.0mm, F.Cu at (163.5, 88.1)
- added TP20: TestPoint, TestPoint:TestPoint_THTPad_2.0x2.0mm_Drill1.0mm, F.Cu at (163.5, 91.1)
- added TP21: TestPoint, TestPoint:TestPoint_THTPad_2.0x2.0mm_Drill1.0mm, F.Cu at (128.8, 76.8)
- added TP22: TestPoint, TestPoint:TestPoint_THTPad_2.0x2.0mm_Drill1.0mm, F.Cu at (128.1, 80.7)
- added Y1: 12MHz, Crystal:Crystal_HC49-U_Vertical, F.Cu at (145.3, 67.6)
- moved U2 79.5 mm to (187.4, 125.5)
- moved U4 13.5 mm to (144.7, 79.6), turned to 180 degrees
Connections:
- U4 pad 1: Net-(U4-Pad1) -> USB_VCC_A
- U4 pad 10: Net-(U4-Pad10) -> USB_DD2_P
- U4 pad 11: Net-(U4-Pad11) -> (no net)
- U4 pad 12: Net-(U4-Pad12) -> USB_VCC_A
- U4 pad 13: Net-(U4-Pad13) -> GND
- U4 pad 14: Net-(U4-Pad14) -> USB_XIN
- U4 pad 15: Net-(U4-Pad15) -> USB_XOUT
- U4 pad 16: Net-(U4-Pad16) -> USB_VCC_A
- U4 pad 17: Net-(U4-Pad17) -> (no net)
- U4 pad 18: Net-(U4-Pad18) -> (no net)
- U4 pad 19: Net-(U4-Pad19) -> (no net)
- U4 pad 2: Net-(U4-Pad2) -> GND
- U4 pad 20: Net-(U4-Pad20) -> GND
- U4 pad 21: Net-(U4-Pad21) -> (no net)
- U4 pad 22: Net-(U4-Pad22) -> (no net)
- U4 pad 23: Net-(U4-Pad23) -> (no net)
- U4 pad 24: Net-(U4-Pad24) -> (no net)
- U4 pad 25: Net-(U4-Pad25) -> (no net)
- U4 pad 26: Net-(U4-Pad26) -> (no net)
- U4 pad 27: Net-(U4-Pad27) -> (no net)
- U4 pad 28: Net-(U4-Pad28) -> (no net)
- U4 pad 29: Net-(U4-Pad29) -> (no net)
- U4 pad 3: Net-(U4-Pad3) -> USB_DIN_N
- U4 pad 30: Net-(U4-Pad30) -> (no net)
- U4 pad 31: Net-(U4-Pad31) -> (no net)
- U4 pad 32: Net-(U4-Pad32) -> (no net)
- U4 pad 33: Net-(U4-Pad33) -> (no net)
- U4 pad 34: Net-(U4-Pad34) -> USB_VCC_D
- U4 pad 35: Net-(U4-Pad35) -> (no net)
- U4 pad 36: Net-(U4-Pad36) -> (no net)
- U4 pad 37: Net-(U4-Pad37) -> (no net)
- U4 pad 38: Net-(U4-Pad38) -> (no net)
- U4 pad 39: Net-(U4-Pad39) -> (no net)
- U4 pad 4: Net-(U4-Pad4) -> USB_DIN_P
- U4 pad 40: Net-(U4-Pad40) -> (no net)
- U4 pad 41: Net-(U4-Pad41) -> (no net)
- U4 pad 42: Net-(U4-Pad42) -> (no net)
- U4 pad 43: Net-(U4-Pad43) -> (no net)
- U4 pad 44: Net-(U4-Pad44) -> (no net)
- U4 pad 45: Net-(U4-Pad45) -> (no net)
- U4 pad 46: Net-(U4-Pad46) -> (no net)
- U4 pad 47: Net-(U4-Pad47) -> +5V
- U4 pad 48: Net-(U4-Pad48) -> (no net)
- U4 pad 5: Net-(U4-Pad5) -> USB_DD1_N
- U4 pad 6: Net-(U4-Pad6) -> USB_DD1_P
- U4 pad 7: Net-(U4-Pad7) -> USB_VCC_A
- U4 pad 8: Net-(U4-Pad8) -> GND
- U4 pad 9: Net-(U4-Pad9) -> USB_DD2_N
