File: raspberry_pi_fan_hat/raspberry_pi_fan_hat/raspberry_pi_fan_hat.kicad_pcb (KiCad board)
At the start: 2 copper layers, 65 x 56 mm, 7 parts, among them J1 Conn_01x02, J2 Conn_01x02, P1 Conn_02x20_Odd_Even

Commit message: Updated for version 1.0
Parts:
- removed J2: Conn_01x02, Connector_PinHeader_2.54mm:PinHeader_1x02_P2.54mm_Horizontal
- added D1: LED_Small, LED_SMD:LED_0805_2012Metric, F.Cu at (209.7, 101.5)
- added D2: LED_Small, LED_SMD:LED_0805_2012Metric, F.Cu at (209.7, 103.6)
- added D3: LED_Small, LED_SMD:LED_0805_2012Metric, F.Cu at (255.1, 101.5)
- added D4: LED_Small, LED_SMD:LED_0805_2012Metric, F.Cu at (255.1, 103.6)
- added G***: LOGO, raspberry_pi_fan_hat:gsd, F.Cu at (213.9, 138.3)
- added R1: R_Small, Resistor_SMD:R_0805_2012Metric, F.Cu at (213.1, 101.5)
- added R2: R_Small, Resistor_SMD:R_0805_2012Metric, F.Cu at (213.1, 103.6)
- added R3: R_Small, Resistor_SMD:R_0805_2012Metric, F.Cu at (251.7, 101.5)
- added R4: R_Small, Resistor_SMD:R_0805_2012Metric, F.Cu at (251.7, 103.6)
- added REF**: OSHW-Logo2_7.3x6mm_SilkScreen, Symbol:OSHW-Logo2_7.3x6mm_SilkScreen, F.Cu at (251.0, 138.3)
- moved J1 18.6 mm to (232.6, 102.3)
Connections:
- P1 pad 27: (no net) -> /ID_SD
- P1 pad 28: (no net) -> /ID_SC
Routing:
- net GND: track 19.1 -> 101.1 mm
- net +3V3: track 0.00 -> 26.7 mm
- net /ID_SC: track 0.00 -> 15.9 mm
- net /ID_SD: track 0.00 -> 10.5 mm
- net +5V: track 31.5 -> 39.9 mm
- net Net-(D2-Pad2): track 0.00 -> 1.55 mm
- net Net-(D1-Pad2): track 0.00 -> 1.55 mm
- net Net-(D4-Pad2): track 0.00 -> 1.55 mm
- net Net-(D3-Pad2): track 0.00 -> 1.55 mm
Other:
- board text added: "(c) akuker 2021"
- board text added: "3.3v"
- board text added: "5v"
- board text added: "GND"
- board text added: "GPIO0"
- board text added: "JLCJLCJLCJLC"
- board text added: "Raspberry Pi Fan Holder v1.0"
- board text added: "https://github.com/akuker/hw_projects"
