File: raspberry_pi_fan_hat/raspberry_pi_fan_hat/raspberry_pi_fan_hat.sch (KiCad schematic (older format))
At the start: 7 parts, among them J1 Conn_01x02, J2 Conn_01x02, P1 Conn_02x20_Odd_Even

Commit message: Updated for version 1.0
Parts:
- removed J2: Conn_01x02, Connector_PinHeader_2.54mm:PinHeader_1x02_P2.54mm_Horizontal, symbol Connector_Generic:Conn_01x02
- added D1, D2, D3, D4: LED_Small, LED_SMD:LED_0805_2012Metric, symbol Device:LED_Small
- added R1, R2, R3, R4: R_Small, Resistor_SMD:R_0805_2012Metric, symbol Device:R_Small
Connections:
- net +3V3: now also R2.1
- net +5V: now also R1.1
- net GND: now also D1.1 (K), D2.1 (K), D3.1 (K), D4.1 (K)
- net ID_SC: now also R4.1
- net ID_SD: now also R3.1
- new net: D1.2 (A), R1.2
- new net: D2.2 (A), R2.2
- new net: D3.2 (A), R3.2
- new net: D4.2 (A), R4.2
- no-connect marks 28 -> 26
Changed lines of the file:
@@
 NoConn ~ 3950 2200
 NoConn ~ 3950 2300
-NoConn ~ 3950 2400
 NoConn ~ 3950 2600
 NoConn ~ 3950 2800
@@
 NoConn ~ 1250 2600
 NoConn ~ 1250 2500
-NoConn ~ 1250 2400
 NoConn ~ 1250 2200
 NoConn ~ 1250 2100
@@
 $EndComp
 $Comp
-L Connector_Generic:Conn_01x02 J2
-U 1 1 60246E75
-P 5300 2000
-F 0 "J2" H 5218 1675 50  0000 C CNN
-F 1 "Conn_01x02" H 5218 1766 50  0000 C CNN
-F 2 "Connector_PinHeader_2.54mm:PinHeader_1x02_P2.54mm_Horizontal" H 5300 2000 50  0001 C CNN
-F 3 "~" H 5300 2000 50  0001 C CNN
-	1    5300 2000
-	-1   0    0    1
-$EndComp
-$Comp
-L power:GND #PWR08
-U 1 1 60246E81
-P 5500 2000
-F 0 "#PWR08" H 5500 1750 50  0001 C CNN
-F 1 "GND" H 5500 1850 50  0000 C CNN
-F 2 "" H 5500 2000 50  0000 C CNN
-F 3 "" H 5500 2000 50  0000 C CNN
-	1    5500 2000
-	1    0    0    -1
-$EndComp
-$Comp
-L power:+5V #PWR07
-U 1 1 60246E7B
-P 5500 1900
-F 0 "#PWR07" H 5500 1750 50  0001 C CNN
-F 1 "+5V" H 5450 2050 50  0000 C CNN
-F 2 "" H 5500 1900 50  0000 C CNN
-F 3 "" H 5500 1900 50  0000 C CNN
-	1    5500 1900
-	1    0    0    -1
-$EndComp
+L Device:R_Small R1
+U 1 1 60561B0E
+P 5900 2950
+F 0 "R1" H 5959 2996 50  0000 L CNN
+F 1 "R_Small" H 5959 2905 50  0000 L CNN
+F 2 "Resistor_SMD:R_0805_2012Metric" H 5900 2950 50  0001 C CNN
+F 3 "~" H 5900 2950 50  0001 C CNN
+	1    5900 2950
+	1    0    0    -1
+$EndComp
+$Comp
+L Device:LED_Small D1
+U 1 1 605620DB
+P 5900 3250
+F 0 "D1" V 5946 3180 50  0000 R CNN
+F 1 "LED_Small" V 5855 3180 50  0000 R CNN
+F 2 "LED_SMD:LED_0805_2012Metric" V 5900 3250 50  0001 C CNN
+F 3 "~" V 5900 3250 50  0001 C CNN
+	1    5900 3250
+	0    -1   -1   0
+$EndComp
+$Comp
+L power:GND #PWR0101
+U 1 1 6056294F
+P 5900 3550
+F 0 "#PWR0101" H 5900 3300 50  0001 C CNN
+F 1 "GND" H 5900 3400 50  0000 C CNN
+F 2 "" H 5900 3550 50  0000 C CNN
+F 3 "" H 5900 3550 50  0000 C CNN
+	1    5900 3550
+	1    0    0    -1
+$EndComp
+$Comp
+L power:+5V #PWR0102
+U 1 1 60563BD0
+P 5900 2750
+F 0 "#PWR0102" H 5900 2600 50  0001 C CNN
+F 1 "+5V" H 5900 2890 50  0000 C CNN
+F 2 "" H 5900 2750 50  0000 C CNN
+F 3 "" H 5900 2750 50  0000 C CNN
+	1    5900 2750
+	1    0    0    -1
+$EndComp
+$Comp
+L power:+3.3V #PWR0103
+U 1 1 60564E9E
+P 6650 2750
+F 0 "#PWR0103" H 6650 2600 50  0001 C CNN
+F 1 "+3.3V" H 6650 2890 50  0000 C CNN
+F 2 "" H 6650 2750 50  0000 C CNN
+F 3 "" H 6650 2750 50  0000 C CNN
+	1    6650 2750
+	1    0    0    -1
+$EndComp
+$Comp
+L Device:R_Small R2
+U 1 1 60566BD1
+P 6650 2950
+F 0 "R2" H 6709 2996 50  0000 L CNN
+F 1 "R_Small" H 6709 2905 50  0000 L CNN
+F 2 "Resistor_SMD:R_0805_2012Metric" H 6650 2950 50  0001 C CNN
+F 3 "~" H 6650 2950 50  0001 C CNN
+	1    6650 2950
+	1    0    0    -1
+$EndComp
+$Comp
+L Device:LED_Small D2
+U 1 1 60566BD7
+P 6650 3250
+F 0 "D2" V 6696 3180 50  0000 R CNN
+F 1 "LED_Small" V 6605 3180 50  0000 R CNN
+F 2 "LED_SMD:LED_0805_2012Metric" V 6650 3250 50  0001 C CNN
+F 3 "~" V 6650 3250 50  0001 C CNN
+	1    6650 3250
+	0    -1   -1   0
+$EndComp
+$Comp
+L power:GND #PWR0104
+U 1 1 60566BDD
+P 6650 3550
+F 0 "#PWR0104" H 6650 3300 50  0001 C CNN
+F 1 "GND" H 6650 3400 50  0000 C CNN
+F 2 "" H 6650 3550 50  0000 C CNN
+F 3 "" H 6650 3550 50  0000 C CNN
+	1    6650 3550
+	1    0    0    -1
+$EndComp
+Wire Wire Line
+	6650 2750 6650 2850
+Wire Wire Line
+	5900 3350 5900 3550
+Wire Wire Line
+	6650 3350 6650 3550
+Wire Wire Line
+	5900 2750 5900 2850
+Wire Wire Line
+	5900 3050 5900 3150
+Wire Wire Line
+	6650 3050 6650 3150
+$Comp
+L Device:R_Small R3
+U 1 1 60571E6B
+P 7400 2950
+F 0 "R3" H 7459 2996 50  0000 L CNN
+F 1 "R_Small" H 7459 2905 50  0000 L CNN
+F 2 "Resistor_SMD:R_0805_2012Metric" H 7400 2950 50  0001 C CNN
+F 3 "~" H 7400 2950 50  0001 C CNN
+	1    7400 2950
+	1    0    0    -1
+$EndComp
+$Comp
+L Device:LED_Small D3
+U 1 1 60571E71
+P 7400 3250
+F 0 "D3" V 7446 3180 50  0000 R CNN
+F 1 "LED_Small" V 7355 3180 50  0000 R CNN
+F 2 "LED_SMD:LED_0805_2012Metric" V 7400 3250 50  0001 C CNN
+F 3 "~" V 7400 3250 50  0001 C CNN
+	1    7400 3250
+	0    -1   -1   0
+$EndComp
+$Comp
+L power:GND #PWR09
+U 1 1 60571E77
+P 7400 3550
+F 0 "#PWR09" H 7400 3300 50  0001 C CNN
+F 1 "GND" H 7400 3400 50  0000 C CNN
+F 2 "" H 7400 3550 50  0000 C CNN
+F 3 "" H 7400 3550 50  0000 C CNN
+	1    7400 3550
+	1    0    0    -1
+$EndComp
+$Comp
+L Device:R_Small R4
+U 1 1 60571E89
+P 8150 2950
+F 0 "R4" H 8209 2996 50  0000 L CNN
+F 1 "R_Small" H 8209 2905 50  0000 L CNN
+F 2 "Resistor_SMD:R_0805_2012Metric" H 8150 2950 50  0001 C CNN
+F 3 "~" H 8150 2950 50  0001 C CNN
+	1    8150 2950
+	1    0    0    -1
+$EndComp
+$Comp
+L Device:LED_Small D4
+U 1 1 60571E8F
+P 8150 3250
+F 0 "D4" V 8196 3180 50  0000 R CNN
+F 1 "LED_Small" V 8105 3180 50  0000 R CNN
+F 2 "LED_SMD:LED_0805_2012Metric" V 8150 3250 50  0001 C CNN
+F 3 "~" V 8150 3250 50  0001 C CNN
+	1    8150 3250
+	0    -1   -1   0
+$EndComp
+$Comp
+L power:GND #PWR010
+U 1 1 60571E95
+P 8150 3550
+F 0 "#PWR010" H 8150 3300 50  0001 C CNN
+F 1 "GND" H 8150 3400 50  0000 C CNN
+F 2 "" H 8150 3550 50  0000 C CNN
+F 3 "" H 8150 3550 50  0000 C CNN
+	1    8150 3550
+	1    0    0    -1
+$EndComp
+Wire Wire Line
+	7400 3350 7400 3550
+Wire Wire Line
+	8150 3350 8150 3550
+Wire Wire Line
+	7400 3050 7400 3150
+Wire Wire Line
+	8150 3050 8150 3150
+Wire Wire Line
+	7400 2650 7400 2850
+Wire Wire Line
+	8150 2650 8150 2850
+Text Label 7400 2650 3    50   ~ 0
+ID_SD
+Text Label 8150 2650 3    50   ~ 0
+ID_SC
 $EndSCHEMATC
