File: scsi_analog_discover_2_board/daisy_chain_board.kicad_pcb (KiCad board)
At the start: 2 copper layers, 65 x 49.8 mm, 59 parts, among them J1 Conn_02x15_Odd_Even, J7 Conn_02x25_Odd_Even, J8 CONFLY DB25, X1 Mac, X2 Dogcow, X3 Mac2, X4 Raspberry Pi, X7 Pi

Commit message: Version 1.0
Parts:
- added J2: Conn_02x15_Odd_Even, Connector_PinHeader_2.54mm:PinHeader_2x15_P2.54mm_Vertical, F.Cu at (188.9, 39.4)
- moved JP22 5.23 mm to (203.3, 58.5), turned to -90 degrees
- moved JP7 5.23 mm to (203.3, 63.8)
- moved J1 2.00 mm to (188.9, 53.7)
- turned JP18 to -90 degrees
- turned JP21 to -90 degrees
- turned JP30 to -90 degrees
Connections:
- net Net-(J1-Pad11) renamed AD2_PIN_11
- net Net-(J1-Pad12) renamed AD2_PIN_12
- net Net-(J1-Pad15) renamed AD2_PIN_15
- net Net-(J1-Pad16) renamed AD2_PIN_16
- net Net-(J1-Pad17) renamed AD2_PIN_17
- net Net-(J1-Pad18) renamed AD2_PIN_18
- net Net-(J1-Pad19) renamed AD2_PIN_19
- net Net-(J1-Pad20) renamed AD2_PIN_20
- net Net-(J1-Pad21) renamed AD2_PIN_21
- net Net-(J1-Pad22) renamed AD2_PIN_22
- net Net-(J1-Pad23) renamed AD2_PIN_23
- net Net-(J1-Pad24) renamed AD2_PIN_24
- net Net-(J1-Pad25) renamed AD2_PIN_25
- net Net-(J1-Pad26) renamed AD2_PIN_26
- net Net-(J1-Pad27) renamed AD2_PIN_27
- net Net-(J1-Pad28) renamed AD2_PIN_28
- net Net-(J1-Pad29) renamed AD2_PIN_29
- net Net-(J1-Pad30) renamed AD2_PIN_30
- net Net-(J1-Pad5) renamed AD2_PIN_5
- net Net-(J1-Pad6) renamed AD2_PIN_6
- J1 pad 1: Net-(J1-Pad1) -> AD2_PIN_1
- J1 pad 10: Net-(J1-Pad10) -> AD2_PIN_10
- J1 pad 13: Net-(J1-Pad13) -> AD2_PIN_13
- J1 pad 14: Net-(J1-Pad14) -> AD2_PIN_14
- J1 pad 2: Net-(J1-Pad2) -> AD2_PIN_2
- J1 pad 3: Net-(J1-Pad3) -> AD2_PIN_3
- J1 pad 4: Net-(J1-Pad4) -> AD2_PIN_4
- J1 pad 7: Net-(J1-Pad7) -> AD2_PIN_7
- J1 pad 8: Net-(J1-Pad8) -> AD2_PIN_8
- J1 pad 9: Net-(J1-Pad9) -> AD2_PIN_9
- JP1 pad 1: (no net) -> AD2_PIN_1
- JP1 pad 2: Net-(J1-Pad1) -> AD2_PIN_1
- JP16 pad 1: Net-(J1-Pad2) -> AD2_PIN_2
- JP16 pad 2: (no net) -> AD2_PIN_2
- JP17 pad 1: Net-(J1-Pad4) -> AD2_PIN_4
- JP17 pad 2: (no net) -> AD2_PIN_4
- JP19 pad 1: Net-(J1-Pad8) -> AD2_PIN_8
- JP19 pad 2: (no net) -> AD2_PIN_8
- JP2 pad 1: (no net) -> AD2_PIN_3
- JP2 pad 2: Net-(J1-Pad3) -> AD2_PIN_3
- JP20 pad 1: Net-(J1-Pad10) -> AD2_PIN_10
- JP20 pad 2: (no net) -> AD2_PIN_10
- JP22 pad 1: Net-(J1-Pad14) -> AD2_PIN_14
- JP22 pad 2: (no net) -> AD2_PIN_14
- JP4 pad 1: (no net) -> AD2_PIN_7
- JP4 pad 2: Net-(J1-Pad7) -> AD2_PIN_7
- JP5 pad 1: (no net) -> AD2_PIN_9
- JP5 pad 2: Net-(J1-Pad9) -> AD2_PIN_9
- JP7 pad 1: (no net) -> AD2_PIN_13
- JP7 pad 2: Net-(J1-Pad13) -> AD2_PIN_13
Routing:
- net GND: track 52.3 -> 165.6 mm, vias 1 -> 7
- net C-D3: track 20.9 -> 81.2 mm, vias 2 -> 4
- net C-D7: track 8.78 -> 63.1 mm, vias 0 -> 2
- net C-D6: track 10.8 -> 64.8 mm, vias 1 -> 3
- net C-D2: track 28.3 -> 82.0 mm, vias 2 -> 4
- net C-D5: track 14.6 -> 67.5 mm, vias 2 -> 4
- net C-D4: track 19.6 -> 72.2 mm, vias 2 -> 4
- net C-D0: track 35.4 -> 85.7 mm, vias 2 -> 4
- net C-D1: track 33.7 -> 83.9 mm, vias 2 -> 4
- net C-I_O: track 25.8 -> 72.5 mm, vias 2 -> 4
- net C-REQ: track 16.3 -> 56.9 mm, vias 2 -> 4
- net C-C_D: track 21.8 -> 56.2 mm, vias 2 -> 4
- net C-BSY: track 15.1 -> 47.4 mm, vias 2 -> 4
- net C-SEL: track 33.3 -> 63.2 mm, vias 2 -> 4
- net AD2_PIN_29: track 0.00 -> 27.6 mm
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Other:
- board size 65 x 49.8 mm -> 65 x 63.1 mm
- net class Default removed
- rule pad_to_mask_clearance: 0.05 -> 0
- board text added: "10"
- board text added: "12"
- board text added: "14"
- board text added: "16"
- board text added: "18"
- board text added: "2"
- board text added: "20"
- board text added: "22"
- board text added: "24"
- board text added: "26"
- board text added: "28"
- board text added: "30"
- board text added: "4"
- board text added: "6"
- board text added: "68kmla Version"
- board text added: "8"
- board text added: "Analog Discovery 2 SCSI Breakout Board"
- board text added: "Analog Discovery 2 breakout board for SCSI Version 1.0"
- board text added: "GND"
- board text removed: "68kmla Version 2.2"
- board text removed: "SCSI Daisy Chain Board"

Commit message: Version 1.0
Routing:
- net AD2_PIN_29: track 27.6 -> 0.00 mm
- net GND: track 165.6 -> 193.2 mm
