File: 12v_buck_converter/12v_buck_converter.kicad_sch (KiCad schematic)
At the start: 20 parts, among them J1 Conn_01x03_Male, J2 Conn_01x03_Male, U1 TPS54331DR

Commit message: Version 1.0
Parts:
- C1, C2: value 4.7u -> (none); footprint Capacitor_SMD:C_0805_2012Metric -> (none)
- C3, C6: value 4.7n -> (none); footprint Capacitor_SMD:C_0805_2012Metric -> (none)
- C4: value 0.1u -> (none); footprint Capacitor_SMD:C_0805_2012Metric -> (none)
- C5: value 0.01u -> (none); footprint Capacitor_SMD:C_0805_2012Metric -> (none)
- C7, C9: value 33u -> (none); footprint Capacitor_SMD:C_0805_2012Metric -> (none)
- C8: value 39p -> (none); footprint Capacitor_SMD:C_0805_2012Metric -> (none); LCSC (none) -> C296098
- D1: value B340A -> (none); footprint Diode_SMD:D_SMA -> (none)
- J1, J2: value Conn_01x03_Male -> (none); footprint Connector_PinHeader_2.54mm:PinHeader_1x03_P2.54mm_Vertical -> (none); LCSC (none) -> DNP
- L1: value 6.8uH -> (none); footprint raspberrypi_supercap_ups_lib:Sunltech_SLO0530H -> (none)
- R1: value 332k -> (none); footprint Resistor_SMD:R_0805_2012Metric -> (none); LCSC (none) -> C17631
- R2: value 68.1k -> (none); footprint Resistor_SMD:R_0805_2012Metric -> (none); LCSC (none) -> C17795
- R3: value 49.9k -> (none); footprint Resistor_SMD:R_0805_2012Metric -> (none); LCSC (none) -> C17719
- R4: value 0 -> (none); footprint Resistor_SMD:R_0805_2012Metric -> (none); LCSC (none) -> C17477
- R5: value 10.2k -> (none); footprint Resistor_SMD:R_0805_2012Metric -> (none); LCSC (none) -> C17402
- R6: value 3.24k -> (none); footprint Resistor_SMD:R_0805_2012Metric -> (none); LCSC (none) -> C17609
- U1: value TPS54331DR -> (none); footprint SOIC127P599X175-8N -> (none)

Commit message: restore values
Parts:
- C1, C2: value (none) -> 4.7u; footprint (none) -> Capacitor_SMD:C_0805_2012Metric
- C3, C6: value (none) -> 4.7n; footprint (none) -> Capacitor_SMD:C_0805_2012Metric
- C4: value (none) -> 0.1u; footprint (none) -> Capacitor_SMD:C_0805_2012Metric
- C5: value (none) -> 0.01u; footprint (none) -> Capacitor_SMD:C_0805_2012Metric
- C7, C9: value (none) -> 33u; footprint (none) -> Capacitor_SMD:C_0805_2012Metric
- C8: value (none) -> 39p; footprint (none) -> Capacitor_SMD:C_0805_2012Metric
- D1: value (none) -> B340A; footprint (none) -> Diode_SMD:D_SMA
- J1, J2: value (none) -> Conn_01x03_Male; footprint (none) -> Connector_PinHeader_2.54mm:PinHeader_1x03_P2.54mm_Vertical
- L1: value (none) -> 6.8uH; footprint (none) -> raspberrypi_supercap_ups_lib:Sunltech_SLO0530H
- R1: value (none) -> 332k; footprint (none) -> Resistor_SMD:R_0805_2012Metric
- R2: value (none) -> 68.1k; footprint (none) -> Resistor_SMD:R_0805_2012Metric
- R3: value (none) -> 49.9k; footprint (none) -> Resistor_SMD:R_0805_2012Metric
- R4: value (none) -> 0; footprint (none) -> Resistor_SMD:R_0805_2012Metric
- R5: value (none) -> 10.2k; footprint (none) -> Resistor_SMD:R_0805_2012Metric
- R6: value (none) -> 3.24k; footprint (none) -> Resistor_SMD:R_0805_2012Metric
- U1: value (none) -> TPS54331DR; footprint (none) -> SOIC127P599X175-8N
Connections:
- net Pre_Inductor_5v: now reaches C4.1, D1.1 (K), L1.1, U1.8 (PH)
