File: scsi_switcher/scsi_switcher.kicad_sch (KiCad schematic)
At the start: 47 parts

Commit message: updates
Parts:
- removed TP1, TP10, TP11, TP12, TP13, TP14, TP15, TP16, TP17, TP18, TP19, TP2, TP20, TP21, TP22, TP23, TP24, TP25, TP3, TP4, TP5, TP6, TP7, TP8, TP9: (no value), symbol Connector:TestPoint_Small
- added H1, H2, H3, H4, H5, H6, H7, H8: (no value), symbol Mechanical:MountingHole
- added J10, J11, J8, J9: (no value), symbol Connector:Conn_01x02_Male
- added J12, J13: (no value), symbol Connector_Generic:Conn_02x25_Odd_Even
Connections:
- net BUTTON_SELECT_0: now also J8.1 (Pin_1)
- net BUTTON_SELECT_1: now also J9.1 (Pin_1)
- net BUTTON_SELECT_2: now also J10.1 (Pin_1)
- net BUTTON_SELECT_3: now also J11.1 (Pin_1)
- net GND: now also J10.2 (Pin_2), J11.2 (Pin_2), J12.1 (Pin_1), J12.11 (Pin_11), J12.13 (Pin_13), J12.15 (Pin_15), J12.17 (Pin_17), J12.19 (Pin_19), J12.21 (Pin_21), J12.23 (Pin_23), J12.27 (Pin_27), J12.29 (Pin_29), J12.3 (Pin_3), J12.31 (Pin_31), J12.33 (Pin_33), J12.35 (Pin_35), J12.37 (Pin_37), J12.39 (Pin_39), J12.41 (Pin_41), J12.43 (Pin_43), J12.45 (Pin_45), J12.47 (Pin_47), J12.49 (Pin_49), J12.5 (Pin_5), J12.7 (Pin_7), J12.9 (Pin_9), J13.1 (Pin_1), J13.11 (Pin_11), J13.13 (Pin_13), J13.15 (Pin_15), J13.17 (Pin_17), J13.19 (Pin_19), J13.21 (Pin_21), J13.23 (Pin_23), J13.27 (Pin_27), J13.29 (Pin_29), J13.3 (Pin_3), J13.31 (Pin_31), J13.33 (Pin_33), J13.35 (Pin_35), J13.37 (Pin_37), J13.39 (Pin_39), J13.41 (Pin_41), J13.43 (Pin_43), J13.45 (Pin_45), J13.47 (Pin_47), J13.49 (Pin_49), J13.5 (Pin_5), J13.7 (Pin_7), J13.9 (Pin_9), J8.2 (Pin_2), J9.2 (Pin_2)
- net J1_Pin10: now also J12.10 (Pin_10), J13.10 (Pin_10)
- net J1_Pin12: now also J12.12 (Pin_12), J13.12 (Pin_12)
- net J1_Pin14: now also J12.14 (Pin_14), J13.14 (Pin_14)
- net J1_Pin16: now also J12.16 (Pin_16), J13.16 (Pin_16)
- net J1_Pin18: now also J12.18 (Pin_18), J13.18 (Pin_18)
- net J1_Pin2: now also J12.2 (Pin_2), J13.2 (Pin_2)
- net J1_Pin20: now also J12.20 (Pin_20), J13.20 (Pin_20)
- net J1_Pin22: now also J12.22 (Pin_22), J13.22 (Pin_22)
- net J1_Pin24: now also J12.24 (Pin_24), J13.24 (Pin_24)
- net J1_Pin26: now also J12.26 (Pin_26), J13.26 (Pin_26)
- net J1_Pin28: now also J12.28 (Pin_28), J13.28 (Pin_28)
- net J1_Pin30: now also J12.30 (Pin_30), J13.30 (Pin_30)
- net J1_Pin32: now also J12.32 (Pin_32), J13.32 (Pin_32)
- net J1_Pin34: now also J12.34 (Pin_34), J13.34 (Pin_34)
- net J1_Pin36: now also J12.36 (Pin_36), J13.36 (Pin_36)
- net J1_Pin38: now also J12.38 (Pin_38), J13.38 (Pin_38)
- net J1_Pin4: now also J12.4 (Pin_4), J13.4 (Pin_4)
- net J1_Pin40: now also J12.40 (Pin_40), J13.40 (Pin_40)
- net J1_Pin42: now also J12.42 (Pin_42), J13.42 (Pin_42)
- net J1_Pin44: now also J12.44 (Pin_44), J13.44 (Pin_44)
- net J1_Pin46: now also J12.46 (Pin_46), J13.46 (Pin_46)
- net J1_Pin48: now also J12.48 (Pin_48), J13.48 (Pin_48)
- net J1_Pin50: now also J12.50 (Pin_50), J13.50 (Pin_50)
- net J1_Pin6: now also J12.6 (Pin_6), J13.6 (Pin_6)
- net J1_Pin8: now also J12.8 (Pin_8), J13.8 (Pin_8)
- net SPARE: now reaches U1.20 (GPIO15)
- net SPARE: now also J6.7 (Pin_7), J7.7 (Pin_7)
- no-connect marks 26 -> 27
Other:
- moved on the sheet: R1, R2, R3, R4, SW1, SW2, SW3, SW4, U1

Commit message: layout draft
Parts:
- removed J10, J11, J8, J9: (no value), symbol Connector:Conn_01x02_Male
- added J9: Conn_02x08_Odd_Even, Connector_PinHeader_2.54mm:PinHeader_2x08_P2.54mm_Vertical, symbol Connector_Generic:Conn_02x08_Odd_Even
- added JP1: SolderJumper_3_Open, Jumper:SolderJumper-3_P1.3mm_Bridged12_RoundedPad1.0x1.5mm, symbol Jumper:SolderJumper_3_Bridged12
- H1, H8: value (none) -> MountingHole; footprint (none) -> MountingHole:MountingHole_2.7mm_M2.5
- H2: renamed from H5; value (none) -> MountingHole; footprint (none) -> MountingHole:MountingHole_2.7mm_M2.5
- H3: renamed from H2; value (none) -> MountingHole; footprint (none) -> MountingHole:MountingHole_2.7mm_M2.5
- H4: renamed from H6; value (none) -> MountingHole; footprint (none) -> MountingHole:MountingHole_2.7mm_M2.5
- H5: renamed from H3; value (none) -> MountingHole; footprint (none) -> MountingHole:MountingHole_2.7mm_M2.5
- H6: renamed from H7; value (none) -> MountingHole; footprint (none) -> MountingHole:MountingHole_2.7mm_M2.5
- H7: renamed from H4; value (none) -> MountingHole; footprint (none) -> MountingHole:MountingHole_2.7mm_M2.5
- J1: renamed from J13; value (none) -> Conn_02x25_Counter_Clockwise; footprint (none) -> Connector_PinHeader_2.54mm:PinHeader_2x25_P2.54mm_Vertical
- J10: renamed from J5; value (none) -> Conn_02x25_Counter_Clockwise; footprint (none) -> Connector_IDC:IDC-Header_2x25_P2.54mm_Vertical
- J2: renamed from J12; value (none) -> Conn_02x25_Counter_Clockwise; footprint (none) -> Connector_PinSocket_2.54mm:PinSocket_2x25_P2.54mm_Vertical
- J3: renamed from J6; value (none) -> Conn_02x06_Odd_Even; footprint (none) -> Connector_PinSocket_2.54mm:PinSocket_2x06_P2.54mm_Vertical
- J4: renamed from J7; value (none) -> Conn_02x06_Odd_Even; footprint (none) -> Connector_PinHeader_2.54mm:PinHeader_2x06_P2.54mm_Vertical
- J5: renamed from J1; value (none) -> Conn_02x25_Counter_Clockwise; footprint (none) -> Connector_IDC:IDC-Header_2x25_P2.54mm_Vertical
- J6: renamed from J2; value (none) -> Conn_02x25_Counter_Clockwise; footprint (none) -> Connector_IDC:IDC-Header_2x25_P2.54mm_Vertical
- J7: renamed from J3; value (none) -> Conn_02x25_Counter_Clockwise; footprint (none) -> Connector_IDC:IDC-Header_2x25_P2.54mm_Vertical
- J8: renamed from J4; value (none) -> Conn_02x25_Counter_Clockwise; footprint (none) -> Connector_IDC:IDC-Header_2x25_P2.54mm_Vertical
- JP2: renamed from JP1; value (none) -> SolderJumper_3_Open; footprint (none) -> Jumper:SolderJumper-3_P1.3mm_Open_RoundedPad1.0x1.5mm
- JP3: renamed from JP2; value (none) -> SolderJumper_3_Open; footprint (none) -> Jumper:SolderJumper-3_P1.3mm_Open_RoundedPad1.0x1.5mm
- JP4: renamed from JP3; value (none) -> SolderJumper_3_Open; footprint (none) -> Jumper:SolderJumper-3_P1.3mm_Open_RoundedPad1.0x1.5mm
- JP5: renamed from JP4; value (none) -> SolderJumper_3_Open; footprint (none) -> Jumper:SolderJumper-3_P1.3mm_Open_RoundedPad1.0x1.5mm
- JP6: renamed from JP5; value (none) -> SolderJumper_3_Open; footprint (none) -> Jumper:SolderJumper-3_P1.3mm_Open_RoundedPad1.0x1.5mm
- JP7: renamed from JP6; value (none) -> SolderJumper_3_Open; footprint (none) -> Jumper:SolderJumper-3_P1.3mm_Open_RoundedPad1.0x1.5mm
- R1, R2, R3, R4: value (none) -> R_Small; footprint (none) -> Resistor_SMD:R_0805_2012Metric
- SW1: value (none) -> SELECT 0; footprint (none) -> Button_Switch_THT:SW_PUSH_6mm
- SW2: value (none) -> SELECT 1; footprint (none) -> Button_Switch_THT:SW_PUSH_6mm
- SW3: value (none) -> SELECT 2; footprint (none) -> Button_Switch_THT:SW_PUSH_6mm
- SW4: value (none) -> SELECT 3; footprint (none) -> Button_Switch_THT:SW_PUSH_6mm
- U1: value (none) -> Pico; footprint (none) -> MCU_RaspberryPi_and_Boards:RPi_Pico_SMD_TH
Connections:
- net +3V3: now also JP1.1 (A)
- net GND: now also J9.1 (Pin_1), J9.11 (Pin_11), J9.13 (Pin_13), J9.15 (Pin_15), J9.3 (Pin_3), J9.5 (Pin_5), J9.7 (Pin_7), J9.9 (Pin_9)
- net GPIO_BUTTON_SELECT_0: now also J9.2 (Pin_2)
- net GPIO_BUTTON_SELECT_1: now also J9.4 (Pin_4)
- net GPIO_BUTTON_SELECT_2: now also J9.6 (Pin_6)
- net GPIO_BUTTON_SELECT_3: now also J9.8 (Pin_8)
- net GPIO_BUTTON_SELECT_4: now also J9.10 (Pin_10)
- net GPIO_BUTTON_SELECT_5: now also J9.12 (Pin_12)
- net GPIO_BUTTON_SELECT_6: now also J9.14 (Pin_14)
- net GPIO_BUTTON_SELECT_7: now also J9.16 (Pin_16)
- net VBUS: now reaches U1.40 (VBUS)
- net VBUS: now also JP1.3 (B)
- new net VDD: JP1.2 (C)
- no-connect marks 27 -> 26

Commit message: graphics updates
Parts:
- added H10, H11: (no value), symbol Mechanical:MountingHole
- added H9: MountingHole, MountingHole:MountingHole_2.7mm_M2.5, symbol Mechanical:MountingHole
Changed lines of the file:
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@@
     (pin "1")
+  )
+  (symbol (lib_id "Mechanical:MountingHole") (at 40.64 27.94 90) (unit 1)
+    (in_bom yes) (on_board yes)
+    (property "Reference" "H9" (id 0) (at 39.37 24.13 90)
+      (effects (font (size 1.27 1.27)) (justify right))
+    )
+    (property "Value" "MountingHole" (id 1) (at 43.18 29.2099 90)
+      (effects (font (size 1.27 1.27)) (justify right) hide)
+    )
+    (property "Footprint" "MountingHole:MountingHole_2.7mm_M2.5" (id 2) (at 40.64 27.94 0)
+      (effects (font (size 1.27 1.27)) hide)
+    )
+    (property "Datasheet" "~" (id 3) (at 40.64 27.94 0)
+      (effects (font (size 1.27 1.27)) hide)
+    )
   )
   (symbol (lib_id "Connector_Generic:Conn_02x25_Odd_Even") (at 60.96 54.61 0) (unit 1)
@@
     (pin "1")
   )
+  (symbol (lib_id "Mechanical:MountingHole") (at 20.32 48.26 90) (unit 1)
+    (in_bom yes) (on_board yes)
+    (property "Reference" "H10" (id 0) (at 19.05 44.45 90)
+      (effects (font (size 1.27 1.27)) (justify right))
+    )
+    (property "Value" "" (id 1) (at 16.51 52.07 90)
+      (effects (font (size 1.27 1.27)) (justify right))
+    )
+    (property "Footprint" "" (id 2) (at 20.32 48.26 0)
+      (effects (font (size 1.27 1.27)) hide)
+    )
+    (property "Datasheet" "~" (id 3) (at 20.32 48.26 0)
+      (effects (font (size 1.27 1.27)) hide)
+    )
+  )
   (symbol (lib_id "power:GND") (at 92.71 102.87 90) (unit 1)
     (in_bom yes) (on_board yes)
@@
     (pin "1")
   )
+  (symbol (lib_id "Mechanical:MountingHole") (at 29.21 48.26 90) (unit 1)
+    (in_bom yes) (on_board yes)
+    (property "Reference" "H11" (id 0) (at 27.94 44.45 90)
+      (effects (font (size 1.27 1.27)) (justify right))
+    )
+    (property "Value" "" (id 1) (at 25.4 52.07 90)
+      (effects (font (size 1.27 1.27)) (justify right))
+    )
+    (property "Footprint" "" (id 2) (at 29.21 48.26 0)
+      (effects (font (size 1.27 1.27)) hide)
+    )
+    (property "Datasheet" "~" (id 3) (at 29.21 48.26 0)
+      (effects (font (size 1.27 1.27)) hide)
+    )
+  )
   (symbol (lib_id "power:GND") (at 151.13 83.82 0) (unit 1)
     (in_bom yes) (on_board yes) (fields_autoplaced)
@@
       (reference "H8") (unit 1) (value "MountingHole") (footprint "MountingHole:MountingHole_2.7mm_M2.5")
     )
+    (path "/12a6a643-8d09-4828-9fdd-0e9da0628c48"
+      (reference "H9") (unit 1) (value "MountingHole") (footprint "MountingHole:MountingHole_2.7mm_M2.5")
+    )
+    (path "/2d0fed17-815d-432f-a7eb-ae8520ef2c33"
+      (reference "H10") (unit 1) (value "CE Logo") (footprint "Symbol:CE-Logo_8.5x6mm_SilkScreen")
+    )
+    (path "/c58fe790-7e21-415d-9f6a-3c1eef576e52"
+      (reference "H11") (unit 1) (value "Kicad Logo") (footprint "Symbol:KiCad-Logo_5mm_Copper")
+    )
     (path "/2014f493-7c21-453d-bb61-dceedb8114da"

Commit message: as ordered... I think
Parts:
- H3: renamed from H10; value (none) -> CE Logo; footprint (none) -> Symbol:CE-Logo_8.5x6mm_SilkScreen
- H6: renamed from H11; value (none) -> Kicad Logo; footprint (none) -> Symbol:KiCad-Logo_5mm_Copper
- R1, R2, R3, R4: value R_Small -> 10k; LCSC (none) -> C17414
- renumbered H8 to H10, H9 to H11, H3 to H4, H4 to H5, H5 to H7, H6 to H8, H7 to H9
Connections:
- net +3V3: now also JP1.3 (B); no longer JP1.1 (A)
- net VBUS: now also JP1.1 (A); no longer JP1.3 (B)
Other:
- added sheet Level_Shifters (Level_Shifters.kicad_sch)
- moved on the sheet: JP1
