File: scsi_switcher/switch_connections.kicad_sch (KiCad schematic)
At the start: 23 parts

Commit message: updates
Changed lines of the file:
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@@
       (effects (font (size 1.27 1.27)) hide)
     )
-    (property "Value" "" (id 1) (at 242.57 41.9099 90)
+    (property "Value" "GND" (id 1) (at 242.57 41.9099 90)
       (effects (font (size 1.27 1.27)) (justify right))
     )
@@
       (effects (font (size 1.27 1.27)) hide)
     )
-    (property "Value" "" (id 1) (at 120.65 90.17 90))
+    (property "Value" "VDD" (id 1) (at 120.65 90.17 90))
     (property "Footprint" "" (id 2) (at 119.38 93.98 0)
       (effects (font (size 1.27 1.27)) hide)
@@
       (effects (font (size 1.27 1.27)) hide)
     )
-    (property "Value" "" (id 1) (at 115.57 93.98 90))
+    (property "Value" "VSS" (id 1) (at 115.57 93.98 90))
     (property "Footprint" "" (id 2) (at 116.84 90.17 0)
       (effects (font (size 1.27 1.27)) hide)
@@
       (effects (font (size 1.27 1.27)) hide)
     )
-    (property "Value" "" (id 1) (at 113.03 93.98 90))
+    (property "Value" "VEE" (id 1) (at 113.03 93.98 90))
     (property "Footprint" "" (id 2) (at 114.3 90.17 0)
       (effects (font (size 1.27 1.27)) hide)

Commit message: layout draft
Parts:
- added C1, C10, C11, C12, C13, C2, C3, C4, C5, C6, C7, C8, C9: 100nF, Capacitor_SMD:C_0805_2012Metric, symbol Device:C_Small
- added J11: Conn_02x04_Odd_Even, Connector_PinHeader_2.54mm:PinHeader_2x04_P2.54mm_Vertical, symbol Connector_Generic:Conn_02x04_Odd_Even
- D1: value (none) -> SEL 0; footprint (none) -> LED_SMD:LED_0805_2012Metric
- D2: value (none) -> SEL 1; footprint (none) -> LED_SMD:LED_0805_2012Metric
- D3: value (none) -> SEL 2; footprint (none) -> LED_SMD:LED_0805_2012Metric
- D4: value (none) -> SEL 3; footprint (none) -> LED_SMD:LED_0805_2012Metric
- JP8: renamed from JP7; value (none) -> SolderJumper_2_Bridged; footprint (none) -> Jumper:SolderJumper-2_P1.3mm_Bridged_RoundedPad1.0x1.5mm
- JP9: renamed from JP8; value (none) -> SolderJumper_2_Bridged; footprint (none) -> Jumper:SolderJumper-2_P1.3mm_Bridged_RoundedPad1.0x1.5mm
- R5, R6, R7, R8: value (none) -> R_Small; footprint (none) -> Resistor_SMD:R_0805_2012Metric
- U10, U11, U12, U13, U14, U2, U3, U4, U5, U6, U7, U8, U9: value (none) -> CD4052B; footprint (none) -> Package_SO:SOIC-16_4.55x10.3mm_P1.27mm
Connections:
- net SEL_LED_0: now also J11.2 (Pin_2)
- net SEL_LED_1: now also J11.4 (Pin_4)
- net SEL_LED_2: now also J11.6 (Pin_6)
- net SEL_LED_3: now also J11.8 (Pin_8)
- net VDD: now also C1.1, C10.1, C11.1, C12.1, C13.1, C2.1, C3.1, C4.1, C5.1, C6.1, C7.1, C8.1, C9.1, J11.1 (Pin_1), J11.3 (Pin_3), J11.5 (Pin_5), J11.7 (Pin_7)
- net VSS: now also C1.2, C10.2, C11.2, C12.2, C13.2, C2.2, C3.2, C4.2, C5.2, C6.2, C7.2, C8.2, C9.2

Commit message: as ordered... I think
Parts:
- D1: value SEL 0 -> Green; LCSC (none) -> C2297
- D2: value SEL 1 -> Green; LCSC (none) -> C2297
- D3: value SEL 2 -> Green; LCSC (none) -> C2297
- D4: value SEL 3 -> Green; LCSC (none) -> C2297
- R5, R6, R7, R8: value R_Small -> 10k; LCSC (none) -> C17414
- U10, U11, U12, U13, U14, U2, U3, U4, U5, U6, U7, U8, U9: footprint Package_SO:SOIC-16_4.55x10.3mm_P1.27mm -> Package_SO:SOP-16_3.9x9.9mm_P1.27mm; LCSC (none) -> C6521
Connections:
- net MUX_INHIBIT renamed MUX_INHIBIT_5V
- net MUX_SELECT_A renamed MUX_SELECT_A_5V
- net MUX_SELECT_B renamed MUX_SELECT_B_5V
