File: VintageKVM/ADB_Video_Port.kicad_sch (KiCad schematic)
At the start: 21 parts, among them J1 DE15_Receptacle_HighDensity_M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

Commit message: started layout
Parts:
- added TP24: TestPoint_Small, TestPoint:TestPoint_Pad_D1.0mm, symbol Connector:TestPoint_Small
Connections:
- net GND: no longer JP6.1 (A)
- new net: JP6.1 (A), TP24.1
Changed lines of the file:
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@@
+    )
+  )
+  (symbol (lib_id "Connector:TestPoint_Small") (at 121.92 38.1 0) (unit 1)
+    (in_bom yes) (on_board yes) (dnp no) (fields_autoplaced)
+    (property "Reference" "TP24" (at 123.19 37.465 0)
+      (effects (font (size 1.27 1.27)) (justify left) hide)
+    )
+    (property "Value" "TestPoint_Small" (at 123.19 40.005 0)
+      (effects (font (size 1.27 1.27)) (justify left) hide)
+    )
+    (property "Footprint" "TestPoint:TestPoint_Pad_D1.0mm" (at 127 38.1 0)
+      (effects (font (size 1.27 1.27)) hide)
+    )
+    (property "Datasheet" "~" (at 127 38.1 0)
+      (effects (font (size 1.27 1.27)) hide)
+    )
+    (property "LCSC" "--" (at 121.92 38.1 0)
+      (effects (font (size 1.27 1.27)) hide)
+    )
+    (pin "1")
+    (instances
+      (project "VintageKVM"
+        (path "/0df57c0f-e3f8-4833-8220-8bc28fb0679b/dc07f00d-46a4-40f3-bf2d-d35802205bc0"
+          (reference "TP24") (unit 1)
+        )
+        (path "/0df57c0f-e3f8-4833-8220-8bc28fb0679b/65bd2f50-e110-43d2-b552-ceb5b0e235fa"
+          (reference "TP25") (unit 1)
+        )
+        (path "/0df57c0f-e3f8-4833-8220-8bc28fb0679b/768c7394-476e-4583-9782-f255c84eb6fd"
+          (reference "TP26") (unit 1)
+        )
+        (path "/0df57c0f-e3f8-4833-8220-8bc28fb0679b/1199b545-6212-4a4f-aca3-94e24cdeabd7"
+          (reference "TP27") (unit 1)
+        )
+        (path "/0df57c0f-e3f8-4833-8220-8bc28fb0679b/b02c78f1-86bc-4a02-8edd-75433b5f5843"
+          (reference "TP28") (unit 1)
+        )
+      )
     )
   )
@@
         )
       )
-    )
-  )
-  (symbol (lib_name "GND_1") (lib_id "power:GND") (at 121.92 38.1 180) (unit 1)
-    (in_bom yes) (on_board yes) (dnp no) (fields_autoplaced)
-    (property "Reference" "#PWR051" (at 121.92 31.75 0)
-      (effects (font (size 1.27 1.27)) hide)
-    )
-    (property "Value" "GND" (at 121.92 34.29 0)
-      (effects (font (size 1.27 1.27)))
-    )
-    (property "Footprint" "" (at 121.92 38.1 0)
-      (effects (font (size 1.27 1.27)) hide)
-    )
-    (property "Datasheet" "" (at 121.92 38.1 0)
-      (effects (font (size 1.27 1.27)) hide)
-    )
-    (pin "1")
-    (instances
-      (project "VintageKVM"
-        (path "/0df57c0f-e3f8-4833-8220-8bc28fb0679b/dc07f00d-46a4-40f3-bf2d-d35802205bc0"
-          (reference "#PWR051") (unit 1)
-        )
-        (path "/0df57c0f-e3f8-4833-8220-8bc28fb0679b/65bd2f50-e110-43d2-b552-ceb5b0e235fa"
-          (reference "#PWR062") (unit 1)
-        )
-        (path "/0df57c0f-e3f8-4833-8220-8bc28fb0679b/768c7394-476e-4583-9782-f255c84eb6fd"
-          (reference "#PWR073") (unit 1)
-        )
-        (path "/0df57c0f-e3f8-4833-8220-8bc28fb0679b/1199b545-6212-4a4f-aca3-94e24cdeabd7"
-          (reference "#PWR084") (unit 1)
-        )
-        (path "/0df57c0f-e3f8-4833-8220-8bc28fb0679b/b02c78f1-86bc-4a02-8edd-75433b5f5843"
-          (reference "#PWR095") (unit 1)
-        )
-      )

Commit message: routing complete
Parts:
- J7: footprint libraries:CUI_MD2-40ST-SMT -> CUI_MD2-40ST-SMT; MF (none) -> CUI Inc; PARTREV (none) -> 1.02; STANDARD (none) -> Manufacturer recommendations
- renumbered TP24 to TP6, TP6 to TP7, TP7 to TP8
