File: VintageKVM/VintageKVM.kicad_pcb (KiCad board)
At the start: 2 copper layers, 164 parts, among them J1 Micro USB, J10 DE15_Receptacle_HighDensity_M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, J12 DE15_Receptacle_HighDensity_M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, J14 DE15_Receptacle_HighDensity_M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, J16 DE15_Receptacle_HighDensity_M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, J4 Conn_02x10_Odd_Even, J5 Conn_01x20_Pin, J6 Conn_01x20_Pin, J8 DE15_Receptacle_HighDensity_M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, Q1 BSS138, Q10 BSS138, Q2 BSS138, Q3 BSS138, Q4 BSS138, Q5 BSS138, Q6 BSS138, Q7 BSS138, Q8 BSS138, Q9 BSS138, U2 TS5V522CPWR, U3 TS5V522CPWR

Commit message: started layout
Parts:
- added C1: 100nF, Capacitor_SMD:C_0402_1005Metric, F.Cu at (183.1, 67.7)
- added C2: 100nF, Capacitor_SMD:C_0402_1005Metric, F.Cu at (84.6, 66.7)
- added TP24: TestPoint_Small, TestPoint:TestPoint_Pad_D1.0mm, B.Cu at (207.3, 59.5)
- added TP25: TestPoint_Small, TestPoint:TestPoint_Pad_D1.0mm, F.Cu at (155.6, 62.8)
- added TP26: TestPoint_Small, TestPoint:TestPoint_Pad_D1.0mm, B.Cu at (107.2, 64.2)
- added TP27: TestPoint_Small, TestPoint:TestPoint_Pad_D1.0mm, B.Cu at (60.1, 62.7)
- added TP28: TestPoint_Small, TestPoint:TestPoint_Pad_D1.0mm, B.Cu at (202.9, 94.2)
- JP1, JP10, JP11, JP12, JP13, JP14, JP15, JP2, JP20, JP21, JP22, JP23, JP24, JP25, JP26, JP27, JP28, JP29, JP3, JP30, JP31, JP32, JP33, JP34, JP39, JP4, JP40, JP41, JP42, JP43, JP44, JP45, JP46, JP47, JP48, JP49, JP5, JP50, JP51, JP52, JP53, JP58, JP59, JP6, JP60, JP61, JP62, JP63, JP64, JP65, JP66, JP67, JP68, JP69, JP7, JP70, JP71, JP72, JP77, JP78, JP79, JP8, JP80, JP81, JP82, JP83, JP84, JP85, JP86, JP87, JP88, JP89, JP9, JP90, JP91, TP10, TP11, TP12, TP13, TP14, TP15, TP16, TP17, TP18, TP19, TP20, TP21, TP22, TP23, TP4, TP5, TP6, TP7, TP8, TP9: moved to B.Cu
- moved JP19 182.1 mm to (235.4, 54.0), turned to 90 degrees
- moved R6 177.3 mm to (235.4, 57.9), turned to 90 degrees
- moved JP18 176.7 mm to (231.1, 54.0), turned to 90 degrees
- moved Q2 171.6 mm to (232.6, 58.9), turned to 90 degrees
- moved R5 171.4 mm to (229.8, 57.9), turned to 90 degrees
- moved JP17 136.9 mm to (226.9, 54.0), turned to 90 degrees
- moved R4 133.3 mm to (228.2, 57.9), turned to 90 degrees
- moved JP16 131.2 mm to (222.6, 54.0), turned to 90 degrees
- moved R3 127.5 mm to (222.6, 57.9), turned to 90 degrees
- moved Q1 126.7 mm to (225.4, 58.9), turned to 90 degrees
- moved JP1 124.3 mm to (217.2, 51.4), turned to 90 degrees
- moved JP3 123.5 mm to (213.6, 51.4), turned to 90 degrees
- moved J7 123.5 mm to (229.0, 44.0), turned to 90 degrees
- moved JP5 123.2 mm to (210.0, 51.4), turned to 90 degrees
- moved JP2 122.2 mm to (215.1, 55.4), turned to 90 degrees
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Connections:
- J4 pad 10: unconnected-(J4-Pin_10-Pad10) -> GND
- J4 pad 7: unconnected-(J4-Pin_7-Pad7) -> GND
- J4 pad 8: unconnected-(J4-Pin_8-Pad8) -> GND
- J6 pad 14: unconnected-(J6-Pin_14-Pad14) -> GPIO21
- J6 pad 4: unconnected-(J6-Pin_4-Pad4) -> 3v3_EN
- JP25 pad 1: GND -> Net-(JP25-A)
- JP44 pad 1: GND -> Net-(JP44-A)
- JP6 pad 1: GND -> Net-(JP6-A)
- JP63 pad 1: GND -> Net-(JP63-A)
- JP82 pad 1: GND -> Net-(JP82-A)
Other:
- board outline added: 200 x 73.6 mm

Commit message: routing complete
Parts:
- removed the JP16 at (222.6, 54.0)
- removed the JP17 at (226.9, 54.0)
- removed the JP18 at (231.1, 54.0)
- removed the JP19 at (235.4, 54.0)
- removed the JP35 at (173.8, 54.0)
- removed the JP36 at (178.1, 54.0)
- removed the JP37 at (182.3, 54.0)
- removed the JP38 at (186.6, 54.0)
- removed the JP54 at (124.9, 54.0)
- removed the JP55 at (129.2, 54.0)
- removed the JP56 at (133.5, 54.0)
- removed the JP57 at (137.8, 54.0)
- removed the JP73 at (76.2, 54.0)
- removed the JP74 at (80.3, 54.0)
- removed the JP75 at (85.1, 54.0)
- removed JP76, JP92, JP93, JP94, JP95: SolderJumper_3_Bridged12, Jumper:SolderJumper-3_P1.3mm_Bridged12_RoundedPad1.0x1.5mm
- removed the R1 at (154.4, 101.8)
- removed the R2 at (150.7, 101.4)
- added TP1: ~, TestPoint:TestPoint_Pad_D1.0mm, B.Cu at (104.0, 104.3)
- added TP2: ~, TestPoint:TestPoint_Pad_D1.0mm, B.Cu at (107.0, 104.3)
- added TP3: ~, TestPoint:TestPoint_Pad_D1.0mm, B.Cu at (110.1, 104.3)
- added U1: Pico, MCU_RaspberryPi_and_Boards:RPi_Pico_SMD_TH, F.Cu at (136.8, 88.1)
- TP11: renamed from TP25; moved to B.Cu
- moved J2 102.1 mm to (154.5, 112.2), turned to 180 degrees
- moved R17 87.3 mm to (172.8, 101.5), turned to -90 degrees
- moved J4 73.0 mm to (119.1, 112.2), turned to 180 degrees
- moved F1 46.7 mm to (110.8, 103.7), turned to 0 degrees
- moved J1 46.3 mm to (106.6, 109.9)
- moved J3 32.0 mm to (237.1, 92.1), turned to 180 degrees
- moved TP24 18.3 mm to (193.9, 94.2), turned to 0 degrees
- moved Q10 15.8 mm to (182.8, 100.5), turned to 90 degrees
- moved JP71 14.3 mm to (210.0, 102.2)
- moved TP27 14.3 mm to (210.0, 94.2), turned to 0 degrees
- moved R20 14.2 mm to (185.6, 101.5), turned to 90 degrees
- moved R19 11.6 mm to (180.0, 101.5), turned to 90 degrees
- moved Q9 7.93 mm to (175.6, 100.5), turned to 90 degrees
- moved U2 6.55 mm to (179.0, 66.5), turned to -90 degrees
- moved TP16 6.07 mm to (110.7, 59.2)
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- renumbered J12 to J10, J13 to J11, J14 to J12, J15 to J13, J16 to J14, J5 to J2, J4 to J3, J6 to J4, J7 to J5, J8 to J6, J9 to J7, J10 to J8, J11 to J9, JP20 to JP16, JP21 to JP17, JP22 to JP18, JP23 to JP19, JP24 to JP20, JP25 to JP21, JP26 to JP22, JP27 to JP23, JP28 to JP24, JP29 to JP25, JP30 to JP26, JP31 to JP27, JP32 to JP28, JP33 to JP29, JP34 to JP30, JP39 to JP31, JP40 to JP32, JP41 to JP33, JP42 to JP34, JP43 to JP35, JP44 to JP36, JP45 to JP37, JP46 to JP38, JP47 to JP39, JP48 to JP40, JP49 to JP41, JP50 to JP42, JP51 to JP43, JP52 to JP44, JP53 to JP45, JP58 to JP46, JP59 to JP47, JP60 to JP48, JP61 to JP49, JP62 to JP50, JP63 to JP51, JP64 to JP52, JP65 to JP53, JP66 to JP54, JP67 to JP55, JP68 to JP56, JP69 to JP57, JP70 to JP58, JP71 to JP59, JP72 to JP60, JP77 to JP61, JP78 to JP62, JP79 to JP63, JP80 to JP64, JP81 to JP65, JP82 to JP66, JP83 to JP67, JP84 to JP68, JP85 to JP69, JP86 to JP70, JP87 to JP71, JP88 to JP72, JP89 to JP73, JP90 to JP74, JP91 to JP75, R4 to R1, R11 to R10, R14 to R11, R13 to R12, R16 to R13, R15 to R14, R18 to R15, R17 to R16, R20 to R17, R19 to R18, R22 to R19, R3 to R2, R21 to R20, R6 to R3, R5 to R4, R8 to R5, R7 to R6, R10 to R7, R9 to R8, R12 to R9, TP9 to TP10, TP10 to TP12, TP11 to TP13, TP12 to TP14, TP13 to TP15, TP26 to TP16, TP14 to TP17, TP15 to TP18, TP16 to TP19, TP17 to TP20, TP27 to TP21, TP18 to TP22, TP19 to TP23, TP20 to TP24, TP21 to TP25, TP28 to TP26, TP22 to TP27, TP23 to TP28, TP24 to TP6, TP6 to TP7, TP7 to TP8, TP8 to TP9
Connections:
- F1 pad 1: Net-(#FLG01-pwr) -> Net-(F1-Pad1)
- J1 pad 5: VBUS -> Net-(F1-Pad1)
- Q1 pad 2: Net-(JP16-C) -> PORT_1_ADB_PWR_ON
- Q1 pad 3: Net-(JP17-C) -> /Input Port 1/ADB_EXT_DATA
- Q10 pad 2: Net-(JP94-C) -> CTRL_PORT_ADB_PWR_ON
- Q10 pad 3: Net-(JP95-C) -> /Control Port/ADB_EXT_DATA
- Q2 pad 2: Net-(JP18-C) -> PORT_1_ADB_DATA
- Q2 pad 3: Net-(JP19-C) -> /Input Port 1/ADB_EXT_PWR_ON
- Q3 pad 2: Net-(JP35-C) -> PORT_2_ADB_PWR_ON
- Q3 pad 3: Net-(JP36-C) -> /Input Port 2/ADB_EXT_DATA
- Q4 pad 2: Net-(JP37-C) -> PORT_2_ADB_DATA
- Q4 pad 3: Net-(JP38-C) -> /Input Port 2/ADB_EXT_PWR_ON
- Q5 pad 2: Net-(JP54-C) -> PORT_3_ADB_PWR_ON
- Q5 pad 3: Net-(JP55-C) -> /Input Port 3/ADB_EXT_DATA
- Q6 pad 2: Net-(JP56-C) -> PORT_3_ADB_DATA
- Q6 pad 3: Net-(JP57-C) -> /Input Port 3/ADB_EXT_PWR_ON
- Q7 pad 2: Net-(JP73-C) -> PORT_4_ADB_PWR_ON
- Q7 pad 3: Net-(JP74-C) -> /Input Port 4/ADB_EXT_DATA
- Q8 pad 2: Net-(JP75-C) -> PORT_4_ADB_DATA
- Q8 pad 3: Net-(JP76-C) -> /Input Port 4/ADB_EXT_PWR_ON
- Q9 pad 2: Net-(JP92-C) -> CTRL_PORT_ADB_DATA
- Q9 pad 3: Net-(JP93-C) -> /Control Port/ADB_EXT_PWR_ON
Routing:
- net +3V3: track 0.00 -> 415.1 mm, vias 0 -> 24
- net CTRL_PORT_RED: track 0.00 -> 229.8 mm, vias 0 -> 5
- net CTRL_PORT_VSYNC: track 0.00 -> 224.1 mm, vias 0 -> 7
- net CTRL_PORT_BLUE: track 0.00 -> 219.9 mm, vias 0 -> 6
- net CTRL_PORT_GREEN: track 0.00 -> 219.3 mm, vias 0 -> 5
- net VBUS: track 0.00 -> 201.7 mm, vias 0 -> 4
- net CTRL_PORT_HSYNC: track 0.00 -> 192.0 mm, vias 0 -> 5
- net PORT_1_ADB_DATA: track 0.00 -> 134.6 mm, vias 0 -> 4
- net I2C0_SCL: track 0.00 -> 132.4 mm, vias 0 -> 1
- net I2C0_SDA: track 0.00 -> 130.7 mm, vias 0 -> 2
- net PORT_1_ADB_PWR_ON: track 0.00 -> 129.2 mm, vias 0 -> 4
- net PORT_4_ADB_PWR_ON: track 0.00 -> 102.5 mm, vias 0 -> 2
- net PORT_4_ADB_DATA: track 0.00 -> 91.8 mm, vias 0 -> 2
- net PORT_2_ADB_PWR_ON: track 0.00 -> 85.0 mm, vias 0 -> 2
- net PORT_2_ADB_DATA: track 0.00 -> 80.0 mm, vias 0 -> 2
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- added copper zone on B.Cu, net GND
- added copper zone on F.Cu, net GND
