File: VintageKVM/VintageKVM.kicad_sch (KiCad schematic)
At the start: 13 parts, among them J12 Micro USB, J2 Conn_02x12_Odd_Even, J4 Conn_02x10_Odd_Even, J5 Conn_01x20_Pin, J6 Conn_01x20_Pin, U1 Pico

Commit message: started layout
Parts:
- renumbered J12 to J1, TP21 to TP1, TP22 to TP2, TP23 to TP3
Changed lines of the file:
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@@
   (symbol (lib_id "Connector:TestPoint_Small") (at 22.86 25.4 0) (unit 1)
     (in_bom yes) (on_board yes) (dnp no)
-    (property "Reference" "TP21" (at 16.51 25.4 0)
+    (property "Reference" "TP1" (at 16.51 25.4 0)
       (effects (font (size 1.27 1.27)) (justify left))
     )
@@
   (symbol (lib_id "Connector:TestPoint_Small") (at 22.86 30.48 0) (unit 1)
     (in_bom yes) (on_board yes) (dnp no)
-    (property "Reference" "TP23" (at 16.51 30.48 0)
+    (property "Reference" "TP3" (at 16.51 30.48 0)
       (effects (font (size 1.27 1.27)) (justify left))
     )
@@
   (symbol (lib_id "Connector:TestPoint_Small") (at 22.86 27.94 0) (unit 1)
     (in_bom yes) (on_board yes) (dnp no)
-    (property "Reference" "TP22" (at 16.51 27.94 0)
+    (property "Reference" "TP2" (at 16.51 27.94 0)
       (effects (font (size 1.27 1.27)) (justify left))
     )
@@
   (symbol (lib_id "SamacSys_Parts:U254-051N-4BH806") (at 22.86 22.86 0) (unit 1)
     (in_bom yes) (on_board yes) (dnp no)
-    (property "Reference" "J12" (at 34.29 16.129 0)
+    (property "Reference" "J1" (at 34.29 16.129 0)
       (effects (font (size 1.27 1.27)))
     )

Commit message: routing complete
Parts:
- removed J2: Conn_02x12_Odd_Even, symbol Connector_Generic:Conn_02x12_Odd_Even
- removed J3: ~, symbol Connector:USB_A
- removed R1, R2: 33, Resistor_SMD:R_0402_1005Metric, symbol Device:R_Small
- J1: footprint libraries:U254051N4BH806 -> U254051N4BH806; Arrow Part Number (none) -> U254-051N-4BH806; Height (none) -> 3
- TP1, TP2, TP3: footprint (none) -> TestPoint:TestPoint_Pad_D1.0mm
- U1: footprint RPi_Pico:RPi_Pico_SMD_TH -> MCU_RaspberryPi_and_Boards:RPi_Pico_SMD_TH
- renumbered J5 to J2, J4 to J3, J6 to J4
Connections:
- net 3v3_EN: now also U1.37 (3V3_EN)
- net GND: no longer U1.42 (GND)
- net GPIO21: now also U1.27 (GPIO21)
- net VBUS: no longer J1.5
- net at F1.1: now also J1.5
- no-connect marks 7 -> 9
Other:
- moved on the sheet: F1, J2, J4, U1
