File: Power_Relay_Pico/disc_io.kicad_sch (KiCad schematic)
At the start: 49 parts, among them J301 External Signals, SW301 SW_Push, SW302 SW_Push, SW303 SW_Push, SW304 SW_Push, SW305 SW_Push, SW306 SW_Push, SW307 SW_Push, SW308 SW_Push, U301 74HC14, U302 74HC595, U303 74HC165, U304 STP08DP05, U305 74HC14, U306 74HC165

Commit message: started routing
Parts:
- removed D301, D302, D303, D304: LED_Small, LED_THT:LED_D3.0mm, symbol Device:LED_Small
- C301, C302, C303, C304, C305, C306, C307, C308: LCSC (none) -> C14663
- J301, JP301, SW301, SW302, SW303, SW304, SW305, SW306, SW307, SW308: LCSC (none) -> --
- R301, R302, R305, R306, R309, R310, R313, R314: LCSC (none) -> C21190
- R303, R304, R307, R308, R311, R312, R315, R316, R318, R319, R320, R321: LCSC (none) -> C25804
