File: Power_Relay_Pico/Power_Relay_Pico.kicad_pcb (KiCad board)
At the start: 2 copper layers, 94 x 54 mm, 103 parts, among them IC1 NCN26010XMNTXG, J1 Ext Power Buttons, J102 Conn_01x02_Pin, J104 Conn_01x02_Pin, J11 DB25_Receptacle, J2 Ext LEDs, J3 Screw_Terminal_01x02, J4 Screw_Terminal_01x02, J5 Screw_Terminal_01x02, J6 Screw_Terminal_01x02, J7 Conn_01x08_Pin, J8 Conn_01x08_Pin, J9 Conn_01x10_Pin, K2 Power 2, K3 Power 3, K4 Power 1, SW1 SW_Push, SW2 SW_Push, SW3 SW_Push, SW4 SW_Push, SW5 SW_Push, SW6 SW_Push, SW7 SW_Push, SW8 SW_Push, SW9 SW_Push, U1 Pico, U2 INA3221, U3 ULN2003, Y1 25MHz, Y2 25MHz

Commit message: start layout
Parts:
- removed C1, C2, C3, C4, C5, C6, C7, C8: 0.1u, Capacitor_SMD:C_0603_1608Metric
- removed J1: Ext Power Buttons, Connector_IDC:IDC-Header_2x08_P2.54mm_Vertical
- removed J102: Conn_01x02_Pin, Connector_PinHeader_2.54mm:PinHeader_1x02_P2.54mm_Vertical
- removed J7, J8: Conn_01x08_Pin, Connector_PinHeader_1.00mm:PinHeader_1x08_P1.00mm_Vertical
- removed R1, R14, R16, R2, R3, R4, R5, R6: 10k, Resistor_SMD:R_0603_1608Metric
- removed R10, R11, R12, R13, R15, R7, R8, R9: 1k, Resistor_SMD:R_0603_1608Metric
- removed SW1, SW2, SW3, SW4, SW5, SW6, SW7, SW8: SW_Push, Button_Switch_THT:SW_PUSH_6mm
- removed U2: INA3221, Package_DFN_QFN:Texas_RGV0016A_VQFN-16-1EP_4x4mm_P0.65mm_EP2.1x2.1mm
- added C301: 0.1u, Capacitor_SMD:C_0603_1608Metric, F.Cu at (58.9, 55.0)
- added C302: 0.1u, Capacitor_SMD:C_0603_1608Metric, F.Cu at (76.0, 55.0)
- added C303: 0.1u, Capacitor_SMD:C_0603_1608Metric, F.Cu at (58.5, 65.0)
- added C304: 0.1u, Capacitor_SMD:C_0603_1608Metric, F.Cu at (75.5, 65.0)
- added C305: 0.1u, Capacitor_SMD:C_0603_1608Metric, F.Cu at (72.6, 55.0)
- added C306: 0.1u, Capacitor_SMD:C_0603_1608Metric, F.Cu at (86.2, 56.1)
- added C307: 0.1u, Capacitor_SMD:C_0603_1608Metric, F.Cu at (72.6, 65.0)
- added C308: 0.1u, Capacitor_SMD:C_0603_1608Metric, F.Cu at (87.0, 61.8)
- added C401: 100n, Capacitor_SMD:C_0603_1608Metric, F.Cu at (94.0, 105.2)
- added C402: 100n, Capacitor_SMD:C_0603_1608Metric, F.Cu at (94.0, 107.7)
- added C403: 100n, Capacitor_SMD:C_0603_1608Metric, F.Cu at (94.0, 110.2)
- added C404: 100n, Capacitor_SMD:C_0603_1608Metric, F.Cu at (94.0, 112.7)
- added C405: 100n, Capacitor_SMD:C_0603_1608Metric, F.Cu at (94.0, 115.2)
- added D301: LED_Small, LED_THT:LED_D3.0mm, F.Cu at (60.0, 73.0)
- added D302: LED_Small, LED_THT:LED_D3.0mm, F.Cu at (69.0, 73.0)
- added D303: LED_Small, LED_THT:LED_D3.0mm, F.Cu at (78.0, 73.0)
- added D304: LED_Small, LED_THT:LED_D3.0mm, F.Cu at (86.0, 73.0)
- added H101: MountingHole, MountingHole:MountingHole_3.2mm_M3, F.Cu at (54.0, 54.0)
- added H102: MountingHole, MountingHole:MountingHole_3.2mm_M3, F.Cu at (146.0, 54.0)
- added H103: MountingHole, MountingHole:MountingHole_3.2mm_M3, F.Cu at (146.0, 146.0)
- added H104: MountingHole, MountingHole:MountingHole_3.2mm_M3, F.Cu at (54.0, 146.0)
- added J12: Conn_01x02_Pin, Connector_PinHeader_2.54mm:PinHeader_1x02_P2.54mm_Vertical, F.Cu at (58.0, 126.5)
- added J13: Conn_01x04_Pin, Connector_PinSocket_2.54mm:PinSocket_1x04_P2.54mm_Vertical, F.Cu at (114.2, 106.3)
- added J301: External Signals, Connector_PinSocket_2.54mm:PinSocket_2x12_P2.54mm_Vertical, F.Cu at (55.0, 63.0)
- added J501: Conn_01x08_Pin, Connector_PinHeader_1.00mm:PinHeader_1x08_P1.00mm_Vertical, F.Cu at (120.1, 105.5)
- added J502: Conn_01x08_Pin, Connector_PinHeader_1.00mm:PinHeader_1x08_P1.00mm_Vertical, F.Cu at (123.5, 105.5)
- added JP102: SolderJumper_2_Open, Jumper:SolderJumper-2_P1.3mm_Open_RoundedPad1.0x1.5mm, F.Cu at (105.3, 105.7)
- added JP103: SolderJumper_2_Open, Jumper:SolderJumper-2_P1.3mm_Open_RoundedPad1.0x1.5mm, F.Cu at (105.3, 109.3)
- added JP104: SolderJumper_2_Open, Jumper:SolderJumper-2_P1.3mm_Open_RoundedPad1.0x1.5mm, F.Cu at (105.3, 112.8)
- added JP105: SolderJumper_2_Open, Jumper:SolderJumper-2_P1.3mm_Open_RoundedPad1.0x1.5mm, F.Cu at (105.3, 116.4)
- added JP106: SolderJumper_2_Open, Jumper:SolderJumper-2_P1.3mm_Open_RoundedPad1.0x1.5mm, F.Cu at (105.3, 119.9)
- added JP107: SolderJumper_2_Open, Jumper:SolderJumper-2_P1.3mm_Open_RoundedPad1.0x1.5mm, F.Cu at (109.7, 105.7)
- added JP108: SolderJumper_2_Open, Jumper:SolderJumper-2_P1.3mm_Open_RoundedPad1.0x1.5mm, F.Cu at (109.7, 109.3)
- added JP109: SolderJumper_2_Open, Jumper:SolderJumper-2_P1.3mm_Open_RoundedPad1.0x1.5mm, F.Cu at (109.7, 112.8)
- added JP301: SolderJumper_2_Bridged, Jumper:SolderJumper-2_P1.3mm_Bridged_RoundedPad1.0x1.5mm, F.Cu at (115.1, 93.3)
- added JP401: SolderJumper_2_Bridged, Jumper:SolderJumper-2_P1.3mm_Bridged_RoundedPad1.0x1.5mm, F.Cu at (85.5, 105.7)
- added JP402: SolderJumper_2_Bridged, Jumper:SolderJumper-2_P1.3mm_Bridged_RoundedPad1.0x1.5mm, F.Cu at (85.5, 109.3)
- added JP403: SolderJumper_2_Bridged, Jumper:SolderJumper-2_P1.3mm_Bridged_RoundedPad1.0x1.5mm, F.Cu at (85.5, 112.8)
- added JP404: SolderJumper_2_Bridged, Jumper:SolderJumper-2_P1.3mm_Bridged_RoundedPad1.0x1.5mm, F.Cu at (85.5, 116.4)
- added JP405: SolderJumper_2_Bridged, Jumper:SolderJumper-2_P1.3mm_Bridged_RoundedPad1.0x1.5mm, F.Cu at (85.5, 119.9)
- added JP406: SolderJumper_2_Bridged, Jumper:SolderJumper-2_P1.3mm_Bridged_RoundedPad1.0x1.5mm, F.Cu at (89.9, 105.7)
- added JP407: SolderJumper_2_Bridged, Jumper:SolderJumper-2_P1.3mm_Bridged_RoundedPad1.0x1.5mm, F.Cu at (89.9, 109.3)
- added JP408: SolderJumper_2_Bridged, Jumper:SolderJumper-2_P1.3mm_Bridged_RoundedPad1.0x1.5mm, F.Cu at (89.9, 112.8)
- added R301: 1k, Resistor_SMD:R_0603_1608Metric, F.Cu at (61.5, 55.0)
- added R302: 1k, Resistor_SMD:R_0603_1608Metric, F.Cu at (70.0, 55.0)
- added R303: 10k, Resistor_SMD:R_0603_1608Metric, F.Cu at (64.1, 55.0)
- added R304: 10k, Resistor_SMD:R_0603_1608Metric, F.Cu at (67.4, 55.0)
- added R305: 1k, Resistor_SMD:R_0603_1608Metric, F.Cu at (78.9, 54.9)
- added R306: 1k, Resistor_SMD:R_0603_1608Metric, F.Cu at (87.5, 54.2)
- added R307: 10k, Resistor_SMD:R_0603_1608Metric, F.Cu at (81.5, 54.9)
- added R308: 10k, Resistor_SMD:R_0603_1608Metric, F.Cu at (128.3, 68.8)
- added R309: 1k, Resistor_SMD:R_0603_1608Metric, F.Cu at (61.3, 65.0)
- added R310: 1k, Resistor_SMD:R_0603_1608Metric, F.Cu at (69.8, 65.0)
- added R311: 10k, Resistor_SMD:R_0603_1608Metric, F.Cu at (64.2, 65.0)
- added R312: 10k, Resistor_SMD:R_0603_1608Metric, F.Cu at (67.0, 65.0)
- added R313: 1k, Resistor_SMD:R_0603_1608Metric, F.Cu at (78.3, 65.0)
- added R314: 1k, Resistor_SMD:R_0603_1608Metric, F.Cu at (86.8, 65.0)
- added R315: 10k, Resistor_SMD:R_0603_1608Metric, F.Cu at (81.1, 65.0)
- added R316: 10k, Resistor_SMD:R_0603_1608Metric, F.Cu at (87.2, 68.3)
- added R317: 5.1k, Resistor_SMD:R_0603_1608Metric, F.Cu at (136.4, 51.2)
- added R318: 10k, Resistor_SMD:R_0603_1608Metric, F.Cu at (136.4, 53.7)
- added R319: 10k, Resistor_SMD:R_0603_1608Metric, F.Cu at (136.4, 56.2)
- added R320: 10k, Resistor_SMD:R_0603_1608Metric, F.Cu at (136.4, 58.7)
- added R321: 10k, Resistor_SMD:R_0603_1608Metric, F.Cu at (136.4, 61.2)
- added SW301: SW_Push, Button_Switch_THT:SW_PUSH_6mm, B.Cu at (63.6, 58.2)
- added SW302: SW_Push, Button_Switch_THT:SW_PUSH_6mm, B.Cu at (72.2, 58.2)
- added SW303: SW_Push, Button_Switch_THT:SW_PUSH_6mm, B.Cu at (80.8, 58.2)
- added SW304: SW_Push, Button_Switch_THT:SW_PUSH_6mm, B.Cu at (89.3, 58.2)
- added SW305: SW_Push, Button_Switch_THT:SW_PUSH_6mm, B.Cu at (63.3, 68.2)
- added SW306: SW_Push, Button_Switch_THT:SW_PUSH_6mm, B.Cu at (72.3, 68.2)
- added SW307: SW_Push, Button_Switch_THT:SW_PUSH_6mm, B.Cu at (80.8, 68.2)
- added SW308: SW_Push, Button_Switch_THT:SW_PUSH_6mm, B.Cu at (89.4, 68.2)
- added U301: 74HC14, Package_SO:SOIC-14_3.9x8.7mm_P1.27mm, F.Cu at (37.2, 79.4)
- added U302: 74HC595, Package_SO:SOIC-16_3.9x9.9mm_P1.27mm, F.Cu at (108.7, 85.8)
- added U303: 74HC165, Package_SO:SOIC-16_3.9x9.9mm_P1.27mm, F.Cu at (117.1, 85.8)
- added U304: STP08DP05, Package_SO:SOIC-16_3.9x9.9mm_P1.27mm, F.Cu at (125.6, 85.8)
- added U305: 74HC14, Package_SO:SOIC-14_3.9x8.7mm_P1.27mm, F.Cu at (108.7, 96.8)
- added U306: 74HC165, Package_SO:SOIC-16_3.9x9.9mm_P1.27mm, F.Cu at (134.0, 85.8)
- added U401: SP3232EET-L, Package_SO:TSSOP-16_4.4x5mm_P0.65mm, F.Cu at (98.4, 118.7)
- added U501: INA3221, Package_DFN_QFN:Texas_RGV0016A_VQFN-16-1EP_4x4mm_P0.65mm_EP2.1x2.1mm, F.Cu at (128.3, 107.1)
- J11: moved to B.Cu
- J2: value Ext LEDs -> DE9_Receptacle; footprint Connector_IDC:IDC-Header_2x04_P2.54mm_Vertical -> Connector_Dsub:DSUB-9_Female_EdgeMount_P2.77mm; moved to F.Cu
- moved J11 211.2 mm to (77.1, 146.0), turned to 180 degrees
- moved D4 204.7 mm to (62.2, 84.1), turned to 180 degrees
- moved J3 190.2 mm to (101.0, 144.0), turned to 180 degrees
- moved R23 173.6 mm to (103.7, 127.2), turned to 90 degrees
- moved L101 169.5 mm to (63.0, 134.0), turned to 90 degrees
- moved J4 167.9 mm to (108.3, 144.0), turned to 180 degrees
- moved K2 166.9 mm to (111.3, 135.8), turned to 90 degrees
- moved TL102 164.0 mm to (59.0, 140.0)
- moved J104 162.7 mm to (54.0, 129.0), turned to 180 degrees
- moved R106 160.0 mm to (54.0, 135.0)
- moved IC1 159.4 mm to (65.1, 128.0)
- moved C109 156.7 mm to (54.0, 137.0)
- moved TL101 156.7 mm to (67.0, 140.0)
- moved J5 155.3 mm to (115.7, 143.9), turned to 180 degrees
- moved R103 154.9 mm to (60.0, 136.0), turned to 90 degrees
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Connections:
- J11 pad 1: unconnected-(J11-Pad1) -> LINEP_OUT
- J11 pad 10: unconnected-(J11-Pad10) -> EXT_DO_4
- J11 pad 11: unconnected-(J11-Pad11) -> EXT_DO_3
- J11 pad 12: unconnected-(J11-Pad12) -> EXT_DO_2
- J11 pad 13: unconnected-(J11-Pad13) -> EXT_DO_1
- J11 pad 14: unconnected-(J11-P14-Pad14) -> LINEN_OUT
- J11 pad 15: unconnected-(J11-P15-Pad15) -> LINEN_OUT
- J11 pad 16: unconnected-(J11-P16-Pad16) -> RS232_2_TX
- J11 pad 17: unconnected-(J11-P17-Pad17) -> RS232_2_RX
- J11 pad 18: unconnected-(J11-P18-Pad18) -> GND
- J11 pad 19: unconnected-(J11-P19-Pad19) -> GND
- J11 pad 2: unconnected-(J11-Pad2) -> LINEP_OUT
- J11 pad 20: unconnected-(J11-P20-Pad20) -> GND
- J11 pad 21: unconnected-(J11-P21-Pad21) -> GND
- J11 pad 22: unconnected-(J11-P22-Pad22) -> GND
- J11 pad 23: unconnected-(J11-P23-Pad23) -> GND
- J11 pad 24: unconnected-(J11-P24-Pad24) -> GND
- J11 pad 25: unconnected-(J11-P25-Pad25) -> GND
- J11 pad 3: unconnected-(J11-Pad3) -> GND
- J11 pad 4: unconnected-(J11-Pad4) -> RS232_1_TX
- J11 pad 5: unconnected-(J11-Pad5) -> RS232_1_RX
- J11 pad 6: unconnected-(J11-Pad6) -> EXT_DI_4
- J11 pad 7: unconnected-(J11-Pad7) -> EXT_DI_3
- J11 pad 8: unconnected-(J11-Pad8) -> EXT_DI_2
- J11 pad 9: unconnected-(J11-Pad9) -> EXT_DI_1
- J2 pad 1: EXT_LED_1 -> PWR_OUT_1
- J2 pad 2: +5V -> PWR_OUT_2
- J2 pad 3: EXT_LED_2 -> PWR_OUT_3
- J2 pad 4: +5V -> GND
- J2 pad 5: EXT_LED_3 -> RELAY_COIL_PWR
- J2 pad 6: +5V -> GND
- J2 pad 7: EXT_LED_4 -> GND
- J2 pad 8: +5V -> GND
- R104 pad 1: Net-(J102-Pin_2) -> LINEP_OUT
- R104 pad 2: Net-(J104-Pin_1) -> Net-(J12-Pin_2)
- U1 pad 10: GPIO_PB_6 -> SR_OUT_EN
- U1 pad 11: GPIO_PB_7 -> UART_2_TX
- U1 pad 12: GPIO_PB_8 -> UART_2_RX
- U1 pad 14: GPIO_LED_1 -> SR_DATA_OUT
- U1 pad 15: GPIO_LED_2 -> unconnected-(U1-GPIO11-Pad15)
- U1 pad 16: GPIO_LED_3 -> UART_1_TX
- U1 pad 17: GPIO_LED_4 -> UART_1_RX
- U1 pad 4: GPIO_PB_1 -> SR_SH_LD
- U1 pad 5: GPIO_PB_2 -> SR_SRCLK
- U1 pad 6: GPIO_PB_3 -> SR_DATA_IN
- U1 pad 7: GPIO_PB_4 -> SR_SRCLK
- U1 pad 9: GPIO_PB_5 -> SR_RCLK
- U3 pad 10: LED_1 -> Net-(JP102-B)
- U3 pad 11: LED_2 -> Net-(JP103-B)
- U3 pad 12: LED_3 -> Net-(JP104-B)
- U3 pad 13: LED_4 -> Net-(JP105-B)
- U3 pad 4: GPIO_LED_1 -> Net-(JP106-A)
- U3 pad 5: GPIO_LED_2 -> Net-(JP107-A)
- U3 pad 6: GPIO_LED_3 -> Net-(JP108-A)
- U3 pad 7: GPIO_LED_4 -> Net-(JP109-A)
Routing:
- net SR_SRCLK: track 0.00 -> 20.9 mm
- net GPIO_PB_4: track 20.9 -> 0.00 mm
- net SPE_RESET: track 0.00 -> 16.6 mm
- net Net-(JP106-A): track 0.00 -> 16.3 mm
- net GPIO_LED_1: track 16.3 -> 0.00 mm
- net LINEP_OUT: track 0.00 -> 15.9 mm
- net LINEN_OUT: track 0.00 -> 15.5 mm
- net Net-(J12-Pin_2): track 0.00 -> 12.3 mm
- net RELAY_COIL_PWR: track 12.2 -> 0.00 mm
- net PWR_OUT_2: track 34.3 -> 46.5 mm
- net EXT_PB_5: track 15.2 -> 27.3 mm
- net Net-(J104-Pin_2): track 0.00 -> 11.2 mm
- net Net-(J104-Pin_1): track 0.00 -> 9.63 mm
- net GND: track 11.8 -> 21.3 mm
- net Net-(JP107-A): track 0.00 -> 9.39 mm
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Other:
- board size 94 x 54 mm -> 100 x 100 mm

Commit message: started routing
Parts:
- removed D1, D2, D3, D301, D302, D303, D304, D4, D5, D6, D7: LED_Small, LED_THT:LED_D3.0mm
- removed J11: DB25_Receptacle, Connector_Dsub:DSUB-25_Female_EdgeMount_P2.77mm
- removed J13: Conn_01x04_Pin, Connector_PinSocket_2.54mm:PinSocket_1x04_P2.54mm_Vertical
- removed J2: DE9_Receptacle, Connector_Dsub:DSUB-9_Female_EdgeMount_P2.77mm
- removed J3, J4, J5, J6: Screw_Terminal_01x02, TerminalBlock:TerminalBlock_Xinya_XY308-2.54-2P_1x02_P2.54mm_Horizontal
- removed JP1: SolderJumper_3_Bridged12, Jumper:SolderJumper-3_P1.3mm_Bridged12_RoundedPad1.0x1.5mm
- removed JP102, JP103, JP104, JP105, JP106, JP107, JP108, JP109: SolderJumper_2_Open, Jumper:SolderJumper-2_P1.3mm_Open_RoundedPad1.0x1.5mm
- removed K2: Power 2, Relay_THT:Relay_SPDT_Hongfa_HF3F-L-xx-1ZL1T
- removed K3: Power 3, Relay_THT:Relay_SPDT_Hongfa_HF3F-L-xx-1ZL1T
- removed K4: Power 1, Relay_THT:Relay_SPDT_Hongfa_HF3F-L-xx-1ZL1T
- removed R17, R18, R19, R20, R24, R25, R26: 1k, Resistor_SMD:R_0603_1608Metric
- removed R21, R22, R23: 0.01, Resistor_SMD:R_1206_3216Metric
- removed U1: Pico, RPi_Pico:RPi_Pico_SMD_TH
- removed U3: ULN2003, Package_SO:SOIC-16_3.9x9.9mm_P1.27mm
- added C501: 0.1u, Capacitor_SMD:C_0603_1608Metric, F.Cu at (137.2, 112.5)
- added D104: LED_Small, LED_SMD:LED_0805_2012Metric, F.Cu at (142.5, 128.9)
- added D105: LED_Small, LED_THT:LED_D3.0mm, B.Cu at (145.0, 129.0)
- added D106: LED_Small, LED_SMD:LED_0805_2012Metric, F.Cu at (142.5, 123.2)
- added D107: LED_Small, LED_THT:LED_D3.0mm, B.Cu at (145.0, 123.2)
- added D108: LED_Small, LED_SMD:LED_0805_2012Metric, F.Cu at (142.5, 117.5)
- added D109: LED_Small, LED_THT:LED_D3.0mm, B.Cu at (145.0, 117.5)
- added D110: LED_Small, LED_THT:LED_D3.0mm, B.Cu at (61.0, 75.3)
- added D111: LED_Small, LED_THT:LED_D3.0mm, B.Cu at (69.7, 75.3)
- added D112: LED_Small, LED_THT:LED_D3.0mm, B.Cu at (78.3, 75.3)
- added D113: LED_Small, LED_THT:LED_D3.0mm, B.Cu at (87.0, 75.3)
- added FB1: FerriteBead_Small, Inductor_SMD:L_0805_2012Metric, F.Cu at (63.4, 121.5)
- added J101: Conn_01x04_Pin, Connector_PinSocket_2.54mm:PinSocket_1x04_P2.54mm_Vertical, F.Cu at (148.0, 60.2)
- added J102: Screw_Terminal_01x02, TerminalBlock:TerminalBlock_Xinya_XY308-2.54-2P_1x02_P2.54mm_Horizontal, B.Cu at (104.3, 146.0)
- added J103: Screw_Terminal_01x02, TerminalBlock:TerminalBlock_Xinya_XY308-2.54-2P_1x02_P2.54mm_Horizontal, B.Cu at (111.9, 146.0)
- added J105: DE9_Receptacle, Connector_Dsub:DSUB-9_Female_EdgeMount_P2.77mm, F.Cu at (134.0, 146.0)
- added J106: Screw_Terminal_01x02, TerminalBlock:TerminalBlock_Xinya_XY308-2.54-2P_1x02_P2.54mm_Horizontal, B.Cu at (119.6, 146.0)
- added J107: Screw_Terminal_01x02, TerminalBlock:TerminalBlock_Xinya_XY308-2.54-2P_1x02_P2.54mm_Horizontal, B.Cu at (145.5, 135.2)
- added J108: DB25_Receptacle, Connector_Dsub:DSUB-25_Female_EdgeMount_P2.77mm, F.Cu at (77.0, 146.0)
- added JP101: SolderJumper_3_Bridged12, Jumper:SolderJumper-3_P1.3mm_Bridged12_RoundedPad1.0x1.5mm, F.Cu at (105.5, 121.0)
- added K101: Power 1, Relay_THT:Relay_SPDT_Hongfa_HF3F-L-xx-1ZL1T, B.Cu at (91.9, 125.1)
- added K102: Power 2, Relay_THT:Relay_SPDT_Hongfa_HF3F-L-xx-1ZL1T, B.Cu at (108.9, 125.1)
- added K103: Power 3, Relay_THT:Relay_SPDT_Hongfa_HF3F-L-xx-1ZL1T, B.Cu at (125.9, 125.1)
- added R113: 10k, Resistor_SMD:R_0603_1608Metric, F.Cu at (67.8, 107.4)
- added R114: 10k, Resistor_SMD:R_0603_1608Metric, F.Cu at (67.8, 109.9)
- added R115: 1k, Resistor_SMD:R_0603_1608Metric, F.Cu at (88.5, 88.0)
- added R116: 1k, Resistor_SMD:R_0603_1608Metric, F.Cu at (73.2, 80.0)
- added R117: 1k, Resistor_SMD:R_0603_1608Metric, F.Cu at (73.2, 82.5)
- added R118: 1k, Resistor_SMD:R_0603_1608Metric, F.Cu at (73.2, 85.0)
- added R119: 1k, Resistor_SMD:R_0603_1608Metric, F.Cu at (73.2, 87.5)
- added R120: 1k, Resistor_SMD:R_0603_1608Metric, F.Cu at (73.2, 90.0)
- added R121: 1k, Resistor_SMD:R_0603_1608Metric, F.Cu at (73.2, 92.5)
- added R122: 0.01, Resistor_SMD:R_1206_3216Metric, F.Cu at (98.0, 130.0)
- added R123: 0.01, Resistor_SMD:R_1206_3216Metric, F.Cu at (115.0, 130.0)
- added R124: 0.01, Resistor_SMD:R_1206_3216Metric, F.Cu at (132.0, 130.0)
- added R501: 250mW 10, Resistor_SMD:R_1206_3216Metric, F.Cu at (95.0, 124.5)
- added R502: 250mW 10, Resistor_SMD:R_1206_3216Metric, F.Cu at (101.0, 124.5)
- added R503: 250mW 10, Resistor_SMD:R_1206_3216Metric, F.Cu at (111.9, 124.5)
- added R504: 250mW 10, Resistor_SMD:R_1206_3216Metric, F.Cu at (117.9, 124.5)
- added R505: 250mW 10, Resistor_SMD:R_1206_3216Metric, F.Cu at (129.0, 124.5)
- added R506: 250mW 10, Resistor_SMD:R_1206_3216Metric, F.Cu at (135.0, 124.5)
- added R507: 20k, Resistor_SMD:R_0603_1608Metric, F.Cu at (95.0, 130.5)
- added R508: 100k, Resistor_SMD:R_0603_1608Metric, F.Cu at (95.0, 128.5)
- added R509: 20k, Resistor_SMD:R_0603_1608Metric, F.Cu at (101.0, 128.5)
- added R510: 20k, Resistor_SMD:R_0603_1608Metric, F.Cu at (112.0, 130.5)
- added R511: 20k, Resistor_SMD:R_0603_1608Metric, F.Cu at (118.0, 128.5)
- added R512: 20k, Resistor_SMD:R_0603_1608Metric, F.Cu at (129.0, 130.5)
- added R513: 20k, Resistor_SMD:R_0603_1608Metric, F.Cu at (135.0, 128.5)
- added R514: 100k, Resistor_SMD:R_0603_1608Metric, F.Cu at (101.0, 130.5)
- added R515: 100k, Resistor_SMD:R_0603_1608Metric, F.Cu at (112.0, 128.5)
- added R516: 100k, Resistor_SMD:R_0603_1608Metric, F.Cu at (118.0, 130.5)
- added R517: 100k, Resistor_SMD:R_0603_1608Metric, F.Cu at (129.0, 128.5)
- added R518: 100k, Resistor_SMD:R_0603_1608Metric, F.Cu at (135.0, 130.5)
- added R519: 10k, Resistor_SMD:R_0603_1608Metric, F.Cu at (126.5, 109.5)
- added R520: 10k, Resistor_SMD:R_0603_1608Metric, F.Cu at (128.2, 109.5)
- added R521: 10k, Resistor_SMD:R_0603_1608Metric, F.Cu at (130.0, 109.5)
- added R522: 10k, Resistor_SMD:R_0603_1608Metric, F.Cu at (130.0, 118.8)
- added R523: 0, Resistor_SMD:R_0603_1608Metric, F.Cu at (137.2, 108.8)
- added R524: 10k, Resistor_SMD:R_0603_1608Metric, F.Cu at (137.2, 110.7)
- added R525: 0, Resistor_SMD:R_0603_1608Metric, F.Cu at (137.2, 107.0)
- added R526: 10k, Resistor_SMD:R_0603_1608Metric, F.Cu at (132.5, 110.5)
- added R527: 10k, Resistor_SMD:R_0603_1608Metric, F.Cu at (133.7, 109.0)
- added U101: Pico, RPi_Pico:RPi_Pico_SMD_TH, B.Cu at (105.0, 76.0)
- added U102: ULN2003, Package_SO:SOIC-16_3.9x9.9mm_P1.27mm, F.Cu at (111.2, 115.5)
- D101, D102, D103: footprint LED_THT:LED_D3.0mm -> LED_SMD:LED_0805_2012Metric
- J501: footprint Connector_PinHeader_1.00mm:PinHeader_1x08_P1.00mm_Vertical -> Connector_PinHeader_2.54mm:PinHeader_1x08_P2.54mm_Vertical
- J502: value Conn_01x08_Pin -> Conn_01x06_Pin; footprint Connector_PinHeader_1.00mm:PinHeader_1x08_P1.00mm_Vertical -> Connector_PinHeader_1.00mm:PinHeader_1x06_P1.00mm_Vertical
- moved SW9 89.0 mm to (52.7, 116.5)
- moved U306 68.7 mm to (65.5, 90.5), turned to 90 degrees
- moved U401 62.9 mm to (142.1, 73.5)
- moved U304 59.7 mm to (66.1, 80.9), turned to 90 degrees
- moved U301 59.5 mm to (75.5, 125.0), turned to -90 degrees
- moved U305 51.2 mm to (76.1, 136.3), turned to -90 degrees
- moved R308 45.7 mm to (84.8, 55.0), turned to 90 degrees
- moved R317 43.8 mm to (178.7, 62.5)
- moved R318 43.8 mm to (178.7, 65.0)
- moved R319 43.8 mm to (178.7, 67.5)
- moved R320 43.8 mm to (178.7, 70.0)
- moved R321 43.8 mm to (178.7, 72.5)
- moved U303 37.3 mm to (80.1, 81.0), turned to 90 degrees
- moved U302 28.7 mm to (80.2, 89.8), turned to 90 degrees
- moved J501 28.2 mm to (146.0, 94.1)
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Connections:
- J501 pad 1: unconnected-(J501-Pin_1-Pad1) -> GND
- J501 pad 2: unconnected-(J501-Pin_2-Pad2) -> +3.3V
- J501 pad 3: unconnected-(J501-Pin_3-Pad3) -> /Current Sense/Address
- J501 pad 4: unconnected-(J501-Pin_4-Pad4) -> GND
- J501 pad 5: unconnected-(J501-Pin_5-Pad5) -> CUR_SENS_TC
- J501 pad 6: unconnected-(J501-Pin_6-Pad6) -> CUR_SENS_WARNING
- J501 pad 7: unconnected-(J501-Pin_7-Pad7) -> CUR_SENS_CRITICAL
- J501 pad 8: unconnected-(J501-Pin_8-Pad8) -> CUR_SENS_PV
- J502 pad 1: unconnected-(J502-Pin_1-Pad1) -> PWR_IN_28V
- J502 pad 2: unconnected-(J502-Pin_2-Pad2) -> PWR_MSR_OUT_1
- J502 pad 3: unconnected-(J502-Pin_3-Pad3) -> PWR_IN_28V
- J502 pad 4: unconnected-(J502-Pin_4-Pad4) -> PWR_MSR_OUT_2
- J502 pad 5: unconnected-(J502-Pin_5-Pad5) -> PWR_IN_28V
- J502 pad 6: unconnected-(J502-Pin_6-Pad6) -> PWR_MSR_OUT_3
- U501 pad 1: unconnected-(U501-IN-3-Pad1) -> Net-(U501-IN-3)
- U501 pad 11: unconnected-(U501-IN-1-Pad11) -> Net-(U501-IN-1)
- U501 pad 12: unconnected-(U501-IN+1-Pad12) -> Net-(U501-IN+1)
- U501 pad 14: unconnected-(U501-IN-2-Pad14) -> Net-(U501-IN-2)
- U501 pad 15: unconnected-(U501-IN+2-Pad15) -> Net-(U501-IN+2)
- U501 pad 16: unconnected-(U501-VPU-Pad16) -> +3.3V
- U501 pad 17: unconnected-(U501-EP-Pad17) -> GND
- U501 pad 2: unconnected-(U501-IN+3-Pad2) -> Net-(U501-IN+3)
- U501 pad 5: unconnected-(U501-A0-Pad5) -> Net-(U501-A0)
Routing:
- net +3.3V: track 6.35 -> 101.8 mm, vias 0 -> 5
- net I2C_SDA: track 5.10 -> 80.0 mm, vias 0 -> 1
- net I2C_SCL: track 5.24 -> 80.0 mm, vias 0 -> 2
- net PWR_IN_28V: track 0.00 -> 74.5 mm
- net GND: track 21.3 -> 70.7 mm, vias 0 -> 1
- net PWR_OUT_1: track 0.00 -> 44.2 mm, vias 0 -> 1
- net Net-(U501-IN+1): track 0.00 -> 41.6 mm, vias 0 -> 2
- net CUR_SENS_TC: track 0.00 -> 39.4 mm, vias 0 -> 3
- net GPIO_RELAY_3: track 39.1 -> 0.00 mm
- net Net-(U501-IN-1): track 0.00 -> 36.9 mm, vias 0 -> 2
- net RELAY_COIL_VCC: track 12.8 -> 47.7 mm
- net GPIO_RELAY_2: track 33.1 -> 0.00 mm
- net GPIO_RELAY_1: track 30.7 -> 0.00 mm
- net Net-(U501-IN+2): track 0.00 -> 26.6 mm, vias 0 -> 2
- net EXT_PB_8: track 26.0 -> 0.00 mm
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- added copper zone on B.Cu, net PWR_IN_28V
- removed copper zone on B.Cu, net PWR_MSR_IN_1
Other:
- outline, holes or cut-outs redrawn

Commit message: as ordered
Parts:
- removed J502: Conn_01x06_Pin, Connector_PinHeader_1.00mm:PinHeader_1x06_P1.00mm_Vertical
- added G***: LOGO, RPi_Pico:straw_hat, B.Cu at (73.2, 87.8)
- added J401: DE9_Receptacle, Connector_Dsub:DSUB-9_Male_EdgeMount_P2.77mm, B.Cu at (134.0, 54.0)
- added REF**: OSHW-Symbol_6.7x6mm_SilkScreen, Symbol:OSHW-Symbol_6.7x6mm_SilkScreen, F.Cu at (58.5, 97.0)
- added TP401: TestPoint_Small, TestPoint:TestPoint_Pad_D1.0mm, B.Cu at (128.5, 57.8)
- added TP402: TestPoint_Small, TestPoint:TestPoint_Pad_D1.0mm, F.Cu at (129.8, 57.8)
- added TP403: TestPoint_Small, TestPoint:TestPoint_Pad_D1.0mm, F.Cu at (132.6, 57.8)
- added TP404: TestPoint_Small, TestPoint:TestPoint_Pad_D1.0mm, F.Cu at (135.4, 57.8)
- added TP405: TestPoint_Small, TestPoint:TestPoint_Pad_D1.0mm, B.Cu at (136.8, 57.8)
- added TP406: TestPoint_Small, TestPoint:TestPoint_Pad_D1.0mm, F.Cu at (138.2, 57.8)
- J101: value Conn_01x04_Pin -> Conn_02x04_Pin; footprint Connector_PinSocket_2.54mm:PinSocket_1x04_P2.54mm_Vertical -> Connector_PinHeader_2.54mm:PinHeader_2x04_P2.54mm_Vertical; moved to B.Cu
- J104, J105, J108, J12, J301, J501, J9, JP401, JP405, R101, R102, SW9, TP102, TP103, TP107: moved to B.Cu
- moved D101 181.1 mm to (52.0, 137.0)
- moved D102 176.6 mm to (52.0, 139.2)
- moved D103 174.9 mm to (52.0, 141.5)
- moved J9 173.5 mm to (53.0, 95.8), turned to 180 degrees
- moved TP103 166.1 mm to (60.2, 133.2), turned to 180 degrees
- moved R109 163.8 mm to (55.5, 139.2), turned to 180 degrees
- moved R110 163.2 mm to (55.5, 137.0), turned to 180 degrees
- moved R112 163.1 mm to (55.5, 141.5), turned to 180 degrees
- moved TP102 160.9 mm to (65.8, 133.2), turned to 180 degrees
- moved TP107 153.8 mm to (72.0, 127.5), turned to 180 degrees
- moved R111 153.0 mm to (64.5, 116.8), turned to 180 degrees
- moved R107 152.8 mm to (60.8, 122.2), turned to -90 degrees
- moved R108 151.1 mm to (62.5, 122.2), turned to 90 degrees
- moved C103 150.8 mm to (54.8, 122.5), turned to 90 degrees
- moved R102 147.6 mm to (62.0, 134.0), turned to 90 degrees
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Connections:
- J101 pad 1: GND -> I2C_SDA
- J101 pad 2: +3.3V -> GND
- J101 pad 4: I2C_SDA -> +3.3V
- U101 pad 19: unconnected-(U101-GPIO14-Pad19)_0 -> SPE_IRQ
- U101 pad 26: unconnected-(U101-GPIO20-Pad26)_0 -> SR_DATA_IN
- U101 pad 27: unconnected-(U101-GPIO21-Pad27)_0 -> SR_SRCLK
- U101 pad 29: unconnected-(U101-GPIO22-Pad29) -> SR_SH_LD
- U101 pad 4: SR_SH_LD -> SPE_SPI_CLK
- U101 pad 5: SR_SRCLK -> MOSI
- U101 pad 6: SR_DATA_IN -> MISO
- U101 pad 7: SR_SRCLK -> SPE_CS
Routing:
- net +3.3V: track 101.8 -> 423.5 mm, vias 5 -> 27
- net +5V: track 0.00 -> 217.6 mm, vias 0 -> 5
- net GND: track 70.7 -> 272.4 mm, vias 1 -> 94
- net SPE_SPI_CLK: track 0.00 -> 159.9 mm, vias 0 -> 5
- net SPE_CS: track 0.00 -> 158.0 mm, vias 0 -> 5
- net RS232_1_TX: track 0.00 -> 151.6 mm, vias 0 -> 6
- net RS232_1_RX: track 0.00 -> 149.3 mm, vias 0 -> 6
- net MOSI: track 0.00 -> 137.2 mm, vias 0 -> 3
- net MISO: track 0.00 -> 132.5 mm, vias 0 -> 3
- net SPE_IRQ: track 0.00 -> 118.5 mm, vias 0 -> 5
- net Net-(JP408-B): track 0.00 -> 89.7 mm, vias 0 -> 6
- net Net-(JP404-A): track 0.00 -> 85.1 mm, vias 0 -> 6
- net SR_RCLK: track 0.00 -> 77.8 mm, vias 0 -> 3
- net Net-(JP407-B): track 0.00 -> 76.3 mm, vias 0 -> 6
- net Net-(JP403-A): track 0.00 -> 75.6 mm, vias 0 -> 6
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Other:
- outline, holes or cut-outs redrawn
- board text added: "BAD WOLF"
- board text added: "JLCJLCJLCJLC"
- board text added: "Pico Power Controller (with SPE) v1 (c)2025 akuker"
