File: Power_Relay_Pico/Power_Relay_Pico.kicad_sch (KiCad schematic)
At the start: 65 parts, among them J1 Ext Power Buttons, J11 DB25_Receptacle, J2 Ext LEDs, J3 Screw_Terminal_01x02, J4 Screw_Terminal_01x02, J5 Screw_Terminal_01x02, J6 Screw_Terminal_01x02, J7 Conn_01x08_Pin, J8 Conn_01x08_Pin, K2 Power 2, K3 Power 3, K4 Power 1, SW1 SW_Push, SW2 SW_Push, SW3 SW_Push, SW4 SW_Push, SW5 SW_Push, SW6 SW_Push, SW7 SW_Push, SW8 SW_Push, U1 Pico, U2 INA3221, U3 ULN2003

Commit message: start layout
Parts:
- removed C1, C2, C3, C4, C5, C6, C7, C8: 0.1u, Capacitor_SMD:C_0603_1608Metric, symbol Device:C_Small
- removed J1: Ext Power Buttons, Connector_IDC:IDC-Header_2x08_P2.54mm_Vertical, symbol Connector_Generic:Conn_02x08_Odd_Even
- removed J2: Ext LEDs, Connector_IDC:IDC-Header_2x04_P2.54mm_Vertical, symbol Connector_Generic:Conn_02x04_Odd_Even
- removed J7, J8: Conn_01x08_Pin, Connector_PinHeader_1.00mm:PinHeader_1x08_P1.00mm_Vertical, symbol Connector:Conn_01x08_Pin
- removed R1, R14, R16, R2, R3, R4, R5, R6: 10k, Resistor_SMD:R_0603_1608Metric, symbol Device:R_Small
- removed R10, R11, R12, R13, R15, R7, R8, R9: 1k, Resistor_SMD:R_0603_1608Metric, symbol Device:R_Small
- removed SW1, SW2, SW3, SW4, SW5, SW6, SW7, SW8: SW_Push, Button_Switch_THT:SW_PUSH_6mm, symbol Switch:SW_Push
- removed U2: INA3221, Package_DFN_QFN:Texas_RGV0016A_VQFN-16-1EP_4x4mm_P0.65mm_EP2.1x2.1mm, symbol Power_Management:INA3221
- added H101, H102, H103, H104: MountingHole, MountingHole:MountingHole_3.2mm_M3, symbol Mechanical:MountingHole
- added J13: Conn_01x04_Pin, Connector_PinSocket_2.54mm:PinSocket_1x04_P2.54mm_Vertical, symbol Connector:Conn_01x04_Pin
- added J2: DE9_Receptacle, Connector_Dsub:DSUB-9_Female_EdgeMount_P2.77mm, symbol Connector:DE9_Receptacle
- added JP102, JP103, JP104, JP105, JP106, JP107, JP108, JP109: SolderJumper_2_Open, Jumper:SolderJumper-2_P1.3mm_Open_RoundedPad1.0x1.5mm, symbol Jumper:SolderJumper_2_Open
Connections:
- net GPIO_PB_4 is gone; now on net SR_SRCLK: U1.7 (GPIO5)
- net +3.3V: now also J13.2 (Pin_2)
- net GND: now also J11.18 (P18), J11.19 (P19), J11.20 (P20), J11.21 (P21), J11.22 (P22), J11.23 (P23), J11.24 (P24), J11.25 (P25), J11.3, J13.1 (Pin_1), J2.4, J2.6, J2.7, J2.8, J2.9
- net GPIO_LED_1: now also JP106.2 (B); no longer U1.14 (GPIO10), U3.4 (I4)
- net GPIO_LED_2: now also JP107.2 (B); no longer U1.15 (GPIO11), U3.5 (I5)
- net GPIO_LED_3: now also JP108.2 (B); no longer U1.16 (GPIO12), U3.6 (I6)
- net GPIO_LED_4: now also JP109.2 (B); no longer U1.17 (GPIO13), U3.7 (I7)
- net I2C_SCL: now also J13.3 (Pin_3)
- net I2C_SDA: now also J13.4 (Pin_4)
- net LED_1: now also JP102.1 (A); no longer U3.10 (O7)
- net LED_2: now also JP103.1 (A); no longer U3.11 (O6)
- net LED_3: now also JP104.1 (A); no longer U3.12 (O5)
- net LED_4: now also JP105.1 (A); no longer U3.13 (O4)
- net PWR_OUT_1: now also J2.1
- net PWR_OUT_2: now also J2.2
- net PWR_OUT_3: now also J2.3
- net RELAY_COIL_PWR: now also J2.5
- net LINEP_OUT: now reaches J11.1
- net LINEP_OUT: now also J11.2
- net EXT_DO_4: now reaches J11.10
- net EXT_DO_3: now reaches J11.11
- net EXT_DO_2: now reaches J11.12
- net EXT_DO_1: now reaches J11.13
- net LINEN_OUT: now reaches J11.14 (P14)
- net LINEN_OUT: now also J11.15 (P15)
- net RS232_2_TX: now reaches J11.16 (P16)
- net RS232_2_RX: now reaches J11.17 (P17)
- net RS232_1_TX: now reaches J11.4
- net RS232_1_RX: now reaches J11.5
- net EXT_DI_4: now reaches J11.6
- net EXT_DI_3: now reaches J11.7
- net EXT_DI_2: now reaches J11.8
- net EXT_DI_1: now reaches J11.9
- net GPIO_PB_1 renamed SR_SH_LD
- net GPIO_PB_2 renamed SR_SRCLK
- net GPIO_PB_3 renamed SR_DATA_IN
- net GPIO_PB_5 renamed SR_RCLK
- net GPIO_PB_6 renamed SR_OUT_EN
- net GPIO_PB_7 renamed UART_2_TX
- net GPIO_PB_8 renamed UART_2_RX
- new net: JP109.1 (A), U3.7 (I7)
- new net: JP103.2 (B), U3.11 (O6)
- new net: JP107.1 (A), U3.5 (I5)
- new net: JP108.1 (A), U3.6 (I6)
- new net: JP105.2 (B), U3.13 (O4)
- new net: JP102.2 (B), U3.10 (O7)
- new net: JP104.2 (B), U3.12 (O5)
- new net: JP106.1 (A), U3.4 (I4)
- new net SR_DATA_OUT: U1.14 (GPIO10)
- new net UART_1_RX: U1.17 (GPIO13)
- new net UART_1_TX: U1.16 (GPIO12)
- no-connect marks 19 -> 20
Other:
- added sheet Current Sense (current_sense.kicad_sch)
- added sheet Discrete IO (disc_io.kicad_sch)
- added sheet RS-232 (RS-232.kicad_sch)
- moved on the sheet: J11

Commit message: started routing
Parts:
- removed JP102, JP103, JP104, JP105, JP106, JP107, JP108, JP109: SolderJumper_2_Open, Jumper:SolderJumper-2_P1.3mm_Open_RoundedPad1.0x1.5mm, symbol Jumper:SolderJumper_2_Open
- added D104, D106, D108: LED_Small, LED_SMD:LED_0805_2012Metric, symbol Device:LED_Small
- added R113, R114: 10k, Resistor_SMD:R_0603_1608Metric, symbol Device:R_Small
- D105: renamed from D5; LCSC (none) -> --
- D107: renamed from D6; LCSC (none) -> --
- D109: renamed from D7; LCSC (none) -> --
- D110: renamed from D1; LCSC (none) -> --
- D111: renamed from D2; LCSC (none) -> --
- D112: renamed from D3; LCSC (none) -> --
- D113: renamed from D4; LCSC (none) -> --
- H101, H102, H103, H104: LCSC (none) -> --
- J101: renamed from J13; LCSC (none) -> --
- J102: renamed from J3; LCSC (none) -> --
- J103: renamed from J4; LCSC (none) -> --
- J105: renamed from J2; LCSC (none) -> --
- J106: renamed from J5; LCSC (none) -> --
- J107: renamed from J6; LCSC (none) -> --
- J108: renamed from J11; LCSC (none) -> --
- JP101: renamed from JP1; LCSC (none) -> --
- K101: renamed from K4; LCSC (none) -> --
- K102: renamed from K2; LCSC (none) -> --
- K103: renamed from K3; LCSC (none) -> --
- R115: renamed from R24; LCSC (none) -> C21190
- R116: renamed from R25; LCSC (none) -> C21190
- R117: renamed from R26; LCSC (none) -> C21190
- R118: renamed from R17; LCSC (none) -> C21190
- R119: renamed from R18; LCSC (none) -> C21190
- R120: renamed from R19; LCSC (none) -> C21190
- R121: renamed from R20; LCSC (none) -> C21190
- U101: renamed from U1; symbol RPi_Pico:Pico -> RPi_Pico_modified:Pico; LCSC (none) -> --
- U102: renamed from U3; LCSC (none) -> C7512
- renumbered R21 to R122, R22 to R123, R23 to R124
Connections:
- net RELAY_COIL_PWR is gone; now on net +28V: J105.5, J107.1 (Pin_1)
- net +3.3V: now also R113.2, R114.2
- net I2C_SCL: now also R113.1
- net I2C_SDA: now also R114.1
- net PWR_OUT_1: now also J105.3; no longer J105.1
- net PWR_OUT_3: now also J105.1; no longer J105.3
- net at D109.1 (K), K101.A1, U102.14 (O3): now also D108.1 (K)
- net at D109.2 (A), R117.1: now also D108.2 (A)
- net at D107.1 (K), K102.A1, U102.15 (O2): now also D106.1 (K)
- net at D105.1 (K), K103.A1, U102.16 (O1): now also D104.1 (K)
- net at D105.2 (A), R115.1: now also D104.2 (A)
- net at D107.2 (A), R116.1: now also D106.2 (A)
- net SR_OUT_EN renamed SR_Output_Enable
- no-connect marks 20 -> 28
Other:
- moved on the sheet: D105, D107, D109, D110, D111, D112, D113, JP101, R115, R116, R117

Commit message: as ordered
Parts:
- removed J101: Conn_01x04_Pin, Connector_PinSocket_2.54mm:PinSocket_1x04_P2.54mm_Vertical, symbol Connector:Conn_01x04_Pin
- added J101: Conn_02x04_Pin, Connector_PinHeader_2.54mm:PinHeader_2x04_P2.54mm_Vertical, symbol Connector_Generic:Conn_02x04_Odd_Even
Connections:
- net +3.3V: now also J101.4 (Pin_4), J101.5 (Pin_5)
- net GND: now also J101.2 (Pin_2), J101.7 (Pin_7)
- net I2C_SCL: now also J101.3 (Pin_3), J101.6 (Pin_6)
- net I2C_SDA: now also J101.1 (Pin_1), J101.8 (Pin_8)
- net SR_DATA_IN: now also U101.26 (GPIO20); no longer U101.6 (GPIO4)
- net SR_SH_LD: now also U101.29 (GPIO22); no longer U101.4 (GPIO2)
- net SR_SRCLK: now also U101.27 (GPIO21); no longer U101.5 (GPIO3), U101.7 (GPIO5)
- net SPE_IRQ: now reaches U101.19 (GPIO14)
- new net MISO: U101.6 (GPIO4)
- new net MOSI: U101.5 (GPIO3)
- new net SPE_CS: U101.7 (GPIO5)
- new net SPE_SPI_CLK: U101.4 (GPIO2)
- no-connect marks 28 -> 23
